File: Kicad Files/FCU_Mainboard_v3.kicad_pcb (KiCad board)
At the start: 2 copper layers, 250 x 100 mm, 131 parts, among them J1 R_OLED, J10 AP2, J11 AP1, J12 BootLoader, J14 ALT_OLED, J15 VSPEED_OLED, J16 R_FD, J17 R_LS, J18 R_CSTR, J19 R_WPT, J2 L_OLED, J20 R_VORD, J21 R_NDB, J22 R_ARPT, J23 LB_PULL, J24 LB_PUSH, J25 LB_hPa/inHg, J26 L_FD, J27 L_LS, J28 L_CSTR, J29 L_WPT, J3 SPD_OLED, J30 SPD/MACH, J31 HDG/TRK, J32 MET_ALT, J33 LVL_OFF, J34 S_PUSH, J35 HDG_ENC, J36 RB_ENC, J37 H_PUSH, J38 RB_PULL, J39 RB_hPa/inHg, J4 HDG_OLED, J40 L_VORD, J41 SPD_ENC, J42 ALT_ENC, J43 A_PUSH, J44 RB_PUSH, J45 A_1H_1K, J46 VS_ENC, J47 L_NDB, J48 VS_PUSH, J49 RVOR/ADF_1, J5 H_T_OLED, J50 RVOR/ADF_2, J51 R_MAP_MODE, J52 L_ARPT, J53 R_MAP_RANGE, J54 L_MAP_MODE, J55 L_MAP_RANGE, J56 LB_ENC, J57 LVOR/ADF_1, J58 LVOR/ADF_2, J6 APPR, J69 S_PULL, J7 EXPED, J70 H_PULL, J71 A_PULL, J72 VS_PULL, J8 LOC, J9 A/THR, P1 USB_C_Plug_USB2.0, SW1 SW_DIP_x03, U1 CD74HC4067M, U2 CD74HC4067M, U3 CD74HC4067M, U4 CD74HC4067M, U5 ATMega2560, U6 CH340G, U7 AMS1117-3.3

Commit message: Fix ERC errors, add VIN netclass, correct P1 value
Housekeeping pass after migrating to KiCad 10. No change to the copper
layout or to the netlist: DRC still reports 0 unconnected items and 0
schematic parity issues.

ERC: 10 violations / 2 errors -> 4 violations / 0 errors

- Remove PWR_FLAG #FLG01 (+5V) and #FLG02 (GND). Both were redundant:
  the USB_B symbol of P1 already declares VBUS and GND as power output
  pins, which is what triggered the pin_to_pin errors. The flags on VIN
  and VCC are kept, those rails are fed by passive connectors (JP1 and
  the ISP header) and would otherwise read as undriven.
- Remove a dangling no-connect flag in the root sheet.
- Add a dedicated VIN netclass: track_width 1.0 mm as the intent for
  future routing, clearance kept at 0.1 mm to match how the rail is
  actually routed. VIN feeds the MCU and the CH340 but matched no
  netclass pattern, so it was falling back to the 0.2 mm default while
  +5V and +3V3 got 1.0 and 0.8 mm.
- Widen a stray 0.601 mm segment on +5V to the class width of 1.0 mm.
  The two 0.4102 mm segments on +3V3 are left alone on purpose: they
  are a deliberate neck to clear the SDA pad of the PCA9548A, and
  widening them breaks clearance against the pad and the GND zone.
- P1 value was USB_C_Plug_USB2.0 while symbol, footprint and silkscreen
  are all USB-B. Corrected to USB_B so the BOM stops lying.

The 120 lib_footprint_mismatch entries still reported by DRC are an
artifact of the KiCad 9 -> 10 library changes, not a design defect.

Co-Authored-By: Claude Opus 5 <noreply@anthropic.com>
Parts:
- P1: value USB_C_Plug_USB2.0 -> USB_B
Changed lines of the file:
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@@
 			)
 		)
-		(property "Value" "USB_C_Plug_USB2.0"
+		(property "Value" "USB_B"
 			(at 6.76 10.27 90)
 			(layer "F.Fab")
@@
 		(start 78.5042 70.85)
 		(end 78.5042 70.9)
-		(width 0.601)
+		(width 1)
 		(layer "F.Cu")
 		(net 18)
