File: Kicad Files/FCU_Mainboard_v3.kicad_pcb (KiCad board)
At the start: 2 copper layers, 250 x 100 mm, 131 parts, among them J1 R_OLED, J10 AP2, J11 AP1, J12 BootLoader, J14 ALT_OLED, J15 VSPEED_OLED, J16 R_FD, J17 R_LS, J18 R_CSTR, J19 R_WPT, J2 L_OLED, J20 R_VORD, J21 R_NDB, J22 R_ARPT, J23 LB_PULL, J24 LB_PUSH, J25 LB_hPa/inHg, J26 L_FD, J27 L_LS, J28 L_CSTR, J29 L_WPT, J3 SPD_OLED, J30 SPD/MACH, J31 HDG/TRK, J32 MET_ALT, J33 LVL_OFF, J34 S_PUSH, J35 HDG_ENC, J36 RB_ENC, J37 H_PUSH, J38 RB_PULL, J39 RB_hPa/inHg, J4 HDG_OLED, J40 L_VORD, J41 SPD_ENC, J42 ALT_ENC, J43 A_PUSH, J44 RB_PUSH, J45 A_1H_1K, J46 VS_ENC, J47 L_NDB, J48 VS_PUSH, J49 RVOR/ADF_1, J5 H_T_OLED, J50 RVOR/ADF_2, J51 R_MAP_MODE, J52 L_ARPT, J53 R_MAP_RANGE, J54 L_MAP_MODE, J55 L_MAP_RANGE, J56 LB_ENC, J57 LVOR/ADF_1, J58 LVOR/ADF_2, J6 APPR, J69 S_PULL, J7 EXPED, J70 H_PULL, J71 A_PULL, J72 VS_PULL, J8 LOC, J9 A/THR, P1 USB_B, SW1 SW_DIP_x03, U1 CD74HC4067M, U2 CD74HC4067M, U3 CD74HC4067M, U4 CD74HC4067M, U5 ATMega2560, U6 CH340G, U7 AMS1117-3.3

Commit message: Add the reservoir capacitors the 3.3V regulator was missing
U7 (AMS1117-3.3) was running without an output capacitor. Its datasheet
lists one as required, not advisory: it is part of the device frequency
compensation. The whole +3V3 net held a single 100nF, and that one is
the PCA9548A decoupler sitting 63 mm away on the other side of the board.

That rail feeds seven OLED displays whose internal charge pumps draw in
pulses, so this is the most likely cause of the freezes the unit shows
in use. An unstable 3.3V rail corrupts I2C, and a corrupted transaction
leaves the Wire library waiting for an ACK that never arrives: the MCU
stays alive but never returns. That matches the symptom, a freeze rather
than a reset, better than a supply brownout does.

  C23  100uF electrolytic   +3V3 - GND   the compensation cap
  C24  100nF ceramic        +3V3 - GND   high frequency
  C21  100uF electrolytic   +5V  - GND   rail reservoir
  C22  100nF ceramic        +5V  - GND   high frequency

Values and footprints follow the RMP V5 board, which uses the same MCU
and the same CH340 with electrolytics at its regulator and has never
frozen. Two boards, one designer, and the one with the capacitors works.

C23 sits 5.6 mm from the regulator output pin, reached by 0.8 mm track.
U7 moved 1 mm and R10 1.5 mm to make room.

C21 ended up 23 mm from the regulator input rather than beside it: there
is no room for a 6.3 mm electrolytic any closer without tearing up the
routing. For an LDO the input capacitor matters far less than the output
one, and it still adds reservoir to a +5V rail that had 400nF in total,
so it was left there. The power section gets laid out properly in the
revision that adds the external supply.

  netlist   198 nets unchanged, 131 -> 135 components, no connection
            altered, no value or footprint changed
  DRC       6 violations, all cosmetic: 2 silkscreen overlaps, 2 silk
            over copper, 2 isolated copper islands
  0 unconnected items, 0 schematic pari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
Parts:
- added C21: 100uF, Capacitor_SMD:C_Elec_6.3x7.7, F.Cu at (95.0, 96.0)
- added C22: 100nF, Capacitor_SMD:C_1206_3216Metric_Pad1.33x1.80mm_HandSolder, F.Cu at (125.0, 112.6)
- added C23: 100uF, Capacitor_SMD:C_Elec_6.3x7.7, F.Cu at (125.9, 101.3)
- added C24: 100nF, Capacitor_SMD:C_1206_3216Metric_Pad1.33x1.80mm_HandSolder, F.Cu at (111.3, 107.1)
- moved R10 1.57 mm to (133.8, 99.7)
- moved U7 1.49 mm to (117.5, 105.0)
Routing:
- net GND: track 64.0 -> 94.0 mm, vias 205 -> 209
- net +3V3: track 494.4 -> 510.4 mm
- net +5V: track 270.3 -> 282.6 mm
- net VIN: track 215.1 -> 223.0 mm
- net UD-: track 38.2 -> 45.3 mm
- net U2_MP_SIG: track 111.2 -> 115.3 mm
- net UD+: track 35.7 -> 39.5 mm
- net MP_S2: track 232.4 -> 231.1 mm
