File: Kicad Files/fcu.kicad_sch (KiCad schematic)
At the start: 23 parts, among them J10 AP2, J11 AP1, J30 SPD/MACH, J31 HDG/TRK, J32 MET_ALT, J33 LVL_OFF, J34 S_PUSH, J35 HDG_ENC, J37 H_PUSH, J41 SPD_ENC, J42 ALT_ENC, J43 A_PUSH, J45 A_1H_1K, J46 VS_ENC, J48 VS_PUSH, J6 APPR, J69 S_PULL, J7 EXPED, J70 H_PULL, J71 A_PULL, J72 VS_PULL, J8 LOC, J9 A/THR

Commit message: Fix ERC errors, add VIN netclass, correct P1 value
Housekeeping pass after migrating to KiCad 10. No change to the copper
layout or to the netlist: DRC still reports 0 unconnected items and 0
schematic parity issues.

ERC: 10 violations / 2 errors -> 4 violations / 0 errors

- Remove PWR_FLAG #FLG01 (+5V) and #FLG02 (GND). Both were redundant:
  the USB_B symbol of P1 already declares VBUS and GND as power output
  pins, which is what triggered the pin_to_pin errors. The flags on VIN
  and VCC are kept, those rails are fed by passive connectors (JP1 and
  the ISP header) and would otherwise read as undriven.
- Remove a dangling no-connect flag in the root sheet.
- Add a dedicated VIN netclass: track_width 1.0 mm as the intent for
  future routing, clearance kept at 0.1 mm to match how the rail is
  actually routed. VIN feeds the MCU and the CH340 but matched no
  netclass pattern, so it was falling back to the 0.2 mm default while
  +5V and +3V3 got 1.0 and 0.8 mm.
- Widen a stray 0.601 mm segment on +5V to the class width of 1.0 mm.
  The two 0.4102 mm segments on +3V3 are left alone on purpose: they
  are a deliberate neck to clear the SDA pad of the PCA9548A, and
  widening them breaks clearance against the pad and the GND zone.
- P1 value was USB_C_Plug_USB2.0 while symbol, footprint and silkscreen
  are all USB-B. Corrected to USB_B so the BOM stops lying.

The 120 lib_footprint_mismatch entries still reported by DRC are an
artifact of the KiCad 9 -> 10 library changes, not a design defect.

Co-Authored-By: Claude Opus 5 <noreply@anthropic.com>
Changed lines of the file:
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@@
-	)
-	(symbol
-		(lib_id "power:PWR_FLAG")
-		(at 41.91 59.69 0)
-		(unit 1)
-		(exclude_from_sim no)
-		(in_bom yes)
-		(on_board yes)
-		(dnp no)
-		(fields_autoplaced yes)
-		(property "Reference" "#FLG02"
-			(at 41.91 57.785 0)
-			(effects
-				(font
-					(size 1.27 1.27)
-				)
-				(hide yes)
-			)
-		)
-		(property "Value" "PWR_FLAG"
-			(at 41.91 54.61 0)
-			(effects
-				(font
-					(size 1.27 1.27)
-				)
-			)
-		)
-		(property "Footprint" ""
-			(at 41.91 59.69 0)
-			(effects
-				(font
-					(size 1.27 1.27)
-				)
-				(hide yes)
-			)
-		)
-		(property "Datasheet" "~"
-			(at 41.91 59.69 0)
-			(effects
-				(font
-					(size 1.27 1.27)
-				)
-				(hide yes)
-			)
-		)
-		(property "Description" "Special symbol for telling ERC where power comes from"
-			(at 41.91 59.69 0)
-			(effects
-				(font
-					(size 1.27 1.27)
-				)
-				(hide yes)
-			)
-		)
-		(pin "1"
-		)
-		(instances
-			(project ""
-				(path "/3267b3f3-6c63-480a-8354-1757ed0a4fd3/52021e17-f88a-4b24-887d-3169c4a17f9c"
-					(reference "#FLG02")
-					(unit 1)
-				)
-			)
-		)
 	)
 	(symbol
