File: Kicad Files/FCU_Mainboard_v3.kicad_sch (KiCad schematic)
At the start: 12 parts, among them U5 ATMega2560

Commit message: Fix ERC errors, add VIN netclass, correct P1 value
Housekeeping pass after migrating to KiCad 10. No change to the copper
layout or to the netlist: DRC still reports 0 unconnected items and 0
schematic parity issues.

ERC: 10 violations / 2 errors -> 4 violations / 0 errors

- Remove PWR_FLAG #FLG01 (+5V) and #FLG02 (GND). Both were redundant:
  the USB_B symbol of P1 already declares VBUS and GND as power output
  pins, which is what triggered the pin_to_pin errors. The flags on VIN
  and VCC are kept, those rails are fed by passive connectors (JP1 and
  the ISP header) and would otherwise read as undriven.
- Remove a dangling no-connect flag in the root sheet.
- Add a dedicated VIN netclass: track_width 1.0 mm as the intent for
  future routing, clearance kept at 0.1 mm to match how the rail is
  actually routed. VIN feeds the MCU and the CH340 but matched no
  netclass pattern, so it was falling back to the 0.2 mm default while
  +5V and +3V3 got 1.0 and 0.8 mm.
- Widen a stray 0.601 mm segment on +5V to the class width of 1.0 mm.
  The two 0.4102 mm segments on +3V3 are left alone on purpose: they
  are a deliberate neck to clear the SDA pad of the PCA9548A, and
  widening them breaks clearance against the pad and the GND zone.
- P1 value was USB_C_Plug_USB2.0 while symbol, footprint and silkscreen
  are all USB-B. Corrected to USB_B so the BOM stops lying.

The 120 lib_footprint_mismatch entries still reported by DRC are an
artifact of the KiCad 9 -> 10 library changes, not a design defect.

Co-Authored-By: Claude Opus 5 <noreply@anthropic.com>
Connections:
- no-connect marks 20 -> 19
Changed lines of the file:
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@@
-	)
-	(no_connect
-		(at 251.46 152.4)
 	)
 	(no_connect

Commit message: Update schematic symbols from KiCad 10 libraries
Ran Update Symbols from Library on all sheets, then repaired two side
effects of it. ERC is now clean: 4 warnings -> 0 violations.

The only change to the netlist in the whole project is the USB shield
pin, which KiCad renamed in both the symbol and the footprint:

  net GND:  P1 pin '5'  ->  P1 pin 'SH'

Everything else is byte-for-byte equivalent electrically: 198 nets, 131
components, 106 nodes on GND, no net added or removed, no Value changed.

Two repairs were needed:

- Update Symbols overwrote the Footprint field of U5 and I2C_1 with the
  library symbol defaults, replacing the custom footprints the board was
  actually built with (U5 would have become Package_QFP:TQFP-100_14x14mm
  _P0.5mm instead of PCM_SFLibrary:TQFP100-0.5-14X14MM, and I2C_1 pointed
  at a library nickname that does not exist). Both restored.
- Device:Crystal_GND24 now stacks its two ground pins at one location
  instead of one above and one below the body. That left a redundant GND
  connection orphaned on each crystal: a global label on XT16MHz1 and a
  power port on XT12MHz1, both removed. Ground still reaches both
  crystals through the connection that remains, which is why the GND net
  is unchanged.

The board file is untouched; updating footprints is a separate step.

Co-Authored-By: Claude Opus 5 <noreply@anthropic.com>
Changed lines of the file:
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@@
-		)
-	)
-	(global_label "GND"
-		(shape input)
-		(at 129.54 166.37 180)
-		(fields_autoplaced yes)
-		(effects
-			(font
-				(size 1.27 1.27)
-			)
-			(justify right)
-		)
-		(property "Intersheetrefs" "${INTERSHEET_REFS}"
-			(at 122.6843 166.37 0)
-			(hide yes)
-			(show_name no)
-			(do_not_autoplace no)
-			(effects
-				(font
-					(size 1.27 1.27)
-				)
-				(justify right)
-			)
 		)
 	)
