File: Kicad Files/efis_left.kicad_sch (KiCad schematic)
At the start: 21 parts, among them J16 R_FD, J17 R_LS, J18 R_CSTR, J19 R_WPT, J20 R_VORD, J21 R_NDB, J22 R_ARPT, J36 RB_ENC, J38 RB_PULL, J39 RB_hPa/inHg, J44 RB_PUSH, J49 RVOR/ADF_1, J50 RVOR/ADF_2, J51 R_MAP_MODE, J53 R_MAP_RANGE, U1 CD74HC4067M, U2 CD74HC4067M

Commit message: Fix ERC errors, add VIN netclass, correct P1 value
Housekeeping pass after migrating to KiCad 10. No change to the copper
layout or to the netlist: DRC still reports 0 unconnected items and 0
schematic parity issues.

ERC: 10 violations / 2 errors -> 4 violations / 0 errors

- Remove PWR_FLAG #FLG01 (+5V) and #FLG02 (GND). Both were redundant:
  the USB_B symbol of P1 already declares VBUS and GND as power output
  pins, which is what triggered the pin_to_pin errors. The flags on VIN
  and VCC are kept, those rails are fed by passive connectors (JP1 and
  the ISP header) and would otherwise read as undriven.
- Remove a dangling no-connect flag in the root sheet.
- Add a dedicated VIN netclass: track_width 1.0 mm as the intent for
  future routing, clearance kept at 0.1 mm to match how the rail is
  actually routed. VIN feeds the MCU and the CH340 but matched no
  netclass pattern, so it was falling back to the 0.2 mm default while
  +5V and +3V3 got 1.0 and 0.8 mm.
- Widen a stray 0.601 mm segment on +5V to the class width of 1.0 mm.
  The two 0.4102 mm segments on +3V3 are left alone on purpose: they
  are a deliberate neck to clear the SDA pad of the PCA9548A, and
  widening them breaks clearance against the pad and the GND zone.
- P1 value was USB_C_Plug_USB2.0 while symbol, footprint and silkscreen
  are all USB-B. Corrected to USB_B so the BOM stops lying.

The 120 lib_footprint_mismatch entries still reported by DRC are an
artifact of the KiCad 9 -> 10 library changes, not a design defect.

Co-Authored-By: Claude Opus 5 <noreply@anthropic.com>
Changed lines of the file:
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@@
-	)
-	(symbol
-		(lib_id "power:PWR_FLAG")
-		(at 247.65 20.32 90)
-		(unit 1)
-		(exclude_from_sim no)
-		(in_bom yes)
-		(on_board yes)
-		(dnp no)
-		(fields_autoplaced yes)
-		(property "Reference" "#FLG01"
-			(at 245.745 20.32 0)
-			(effects
-				(font
-					(size 1.27 1.27)
-				)
-				(hide yes)
-			)
-		)
-		(property "Value" "PWR_FLAG"
-			(at 243.84 20.3199 90)
-			(effects
-				(font
-					(size 1.27 1.27)
-				)
-				(justify left)
-			)
-		)
-		(property "Footprint" ""
-			(at 247.65 20.32 0)
-			(effects
-				(font
-					(size 1.27 1.27)
-				)
-				(hide yes)
-			)
-		)
-		(property "Datasheet" "~"
-			(at 247.65 20.32 0)
-			(effects
-				(font
-					(size 1.27 1.27)
-				)
-				(hide yes)
-			)
-		)
-		(property "Description" "Special symbol for telling ERC where power comes from"
-			(at 247.65 20.32 0)
-			(effects
-				(font
-					(size 1.27 1.27)
-				)
-				(hide yes)
-			)
-		)
-		(pin "1"
-		)
-		(instances
-			(project ""
-				(path "/3267b3f3-6c63-480a-8354-1757ed0a4fd3/7bf10440-422c-440c-bb91-38e3488d557b"
-					(reference "#FLG01")
-					(unit 1)
-				)
-			)
-		)
 	)
 	(symbol
