File: PSU/9V_Distribution.kicad_pcb (KiCad board)
At the start: 2 copper layers, 50 x 70 mm, 20 parts, among them J1 Screw_Terminal_2_P5.00mm, J2 Screw_Terminal_2_P5.00mm, J3 Screw_Terminal_2_P5.00mm, J4 Screw_Terminal_2_P5.00mm, U4 LM2596S-5

Commit message: Give the PSU buck the catch diode it never had
The LM2596 on the 9V distribution board has been running without a
freewheel diode. Net-(U4-OUT) held exactly two nodes, U4.2 and L1.1: the
only Schottky on the board is D1, in series at the input as reverse
protection. With nowhere else to go, the inductor current has been
freewheeling through the regulator's own substrate diode, adding roughly
0.4 W inside the package on top of its own 0.7 W. That is why the board
works, and why it wears out.

  D2  SS54 Schottky, cathode on the switch node, anode to ground.
  C4  220uF electrolytic beside C2, to give the control loop the ESR a
      ceramic output capacitor does not provide.
  F2  MF-RHT100 -> MF-RHT200. The input draws ~0.75 A and a 1 A polyfuse
      derates below 0.8 A in a warm printed case. Identical pads.

The power section is re-laid out around this. U4 pin 2, D2's cathode and
L1 pin 1 now sit on one straight line at y=64.95, and C1 moved under the
VIN pin, flipped so its ground terminal faces D2's anode. Every track is
on the front, so the bottom stays an uninterrupted ground plane and each
loop's return runs directly beneath its outward track. Stitching vias at
the ground terminals connect to their pads by track, not through thermal
spokes.

Outline, mounting holes and J1-J4 are untouched: same case, same wiring.

0 unconnected items, 0 schematic parity issues. DRC still reports the
stale ground pour until the zone is refilled in Pcbnew; with the fill
polygons stripped, clearance, hole and solder-mask checks are all clean
and only the pre-existing missing-library warnings remain.

The board in service is still the old one. The Readme says what to bodge
onto it in the meantime.

Co-Authored-By: Claude Opus 5 <noreply@anthropic.com>
Parts:
- added C4: 220uF, Capacitor_THT:CP_Radial_D6.3mm_P2.50mm, F.Cu at (140.0, 76.5)
- added D2: SS54, PCM_Diode_SMD_AKL:D_SMC, F.Cu at (126.0, 68.3)
- F2: value Polyfuse -> 2A; footprint Fuse:Fuse_Bourns_MF-RHT100 -> Fuse:Fuse_Bourns_MF-RHT200
- moved F2 32.6 mm to (104.5, 71.0)
- moved D1 28.0 mm to (110.0, 79.0)
- moved C2 20.9 mm to (134.0, 74.5)
- moved L1 8.96 mm to (135.0, 65.0)
- moved C1 3.91 mm to (119.0, 70.6), turned to 180 degrees
Routing:
- net Net-(LED1-A): track 123.8 -> 160.7 mm
- net Net-(U4-VIN): track 32.1 -> 16.7 mm
- net GND: track 2.00 -> 10.5 mm, vias 15 -> 17
- net Net-(D2-K): track 9.28 -> 15.3 mm
- net Net-(D1-A): track 18.4 -> 12.4 mm
- net Net-(D1-K): track 6.82 -> 3.00 mm
