File: PSU/9V_Distribution.kicad_pcb (KiCad board)
At the start: 2 copper layers, 70 x 80 mm, 29 parts, among them J1 Screw_Terminal_2_P5.00mm, J2 Screw_Terminal_2_P5.00mm, J3 Screw_Terminal_2_P5.00mm, J4 Screw_Terminal_2_P5.00mm, J5 Screw_Terminal_2_P5.00mm, U1 P78A05-1000, U4 LM2596S-5

Commit message: Say on the silkscreen what plugs into each connector
Le schede da fabbricate non si leggevano: quasi tutti i valori stavano su
F.Fab, che non va in stampa, e meta' dei connettori aveva come nome il tipo
di morsetto invece di cosa ci va attaccato.

Nessun valore e' stato riscritto: il nome del componente resta quello che
dice KiCad. Si e' lavorato solo sul serigrafico, in due modi.

I valori che gia' dicono qualcosa di utile sono passati su F.Silk, cosi' si
stampano: Backlighting POT sul dimmer, BTN+LED e BK_LED sui Korry, e i 220 e
91 delle due resistenze, che da montare sono due rettangoli identici.

Dove il valore e' il tipo di morsetto e stampalo non servirebbe a niente, il
valore resta dov'e' e accanto ci va una scritta che dice dove va il filo:

  PSU        J1 -> 9V IN, J2/J3/J4 -> 5V BACKLIGHT, J5 -> 5V MAINBOARD
  Dimmer     J32 -> 5V IN, J12/J13/J14 -> TO LEDMODULE
  LEDModule  J11 -> 5V IN

Ogni posizione e' stata verificata contro pad, altre scritte, contorni
serigrafici e bordo scheda, e poi ricontrollata col DRC, che e' l'unico a
sapere quanto e' larga davvero l'apertura di maschera di un foro di
fissaggio: la scritta di J14 ci finiva sopra, e il valore di J1 sul Korry
grande finiva a cavallo del bordo.

Tutte e cinque le schede: 0 scollegamenti, 0 differenze con lo schema,
nessuna violazione serigrafica. Restano solo gli avvisi di libreria.

Co-Authored-By: Claude Opus 5 <noreply@anthropic.com>
Other:
- board text added: "5V BACKLIGHT"
- board text added: "5V MAINBOARD"
- board text added: "9V IN"
Changed lines of the file:
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@@
 	)
 	(embedded_fonts no)
+	(gr_text "5V BACKLIGHT"
+		(at 109.5 24 0)
+		(layer "F.SilkS")
+		(effects
+			(font
+				(size 1 1)
+				(thickness 0.15)
+			)
+		)
+	)
+	(gr_text "5V BACKLIGHT"
+		(at 125 24 0)
+		(layer "F.SilkS")
+		(effects
+			(font
+				(size 1 1)
+				(thickness 0.15)
+			)
+		)
+	)
+	(gr_text "5V BACKLIGHT"
+		(at 140.5 24 0)
+		(layer "F.SilkS")
+		(effects
+			(font
+				(size 1 1)
+				(thickness 0.15)
+			)
+		)
+	)
+	(gr_text "5V MAINBOARD"
+		(at 157.5 25.5 0)
+		(layer "F.SilkS")
+		(effects
+			(font
+				(size 1 1)
+				(thickness 0.15)
+			)
+		)
+	)
+	(gr_text "9V IN"
+		(at 140.5 97 0)
+		(layer "F.SilkS")
+		(effects
+			(font
+				(size 1 1)
+				(thickness 0.15)
+			)
+		)
+	)
 )

Commit message: Give the 9 V rail a name
La classe di rete da 1.0 mm cercava una rete chiamata +9V che non esisteva:
il ramo dei 9 V non aveva nome e si chiamava Net-(D1-A), Net-(D1-K),
Net-(U4-VIN). Quindi la classe non prendeva niente, e una pista nuova su
quel ramo sarebbe uscita da 0.2 mm, la larghezza del Default. Il ramo della
mainboard un nome ce l'aveva gia', VIN_MB; questo no.

Tre etichette sui fili che c'erano gia', nello stile delle altre del foglio:

  9V_IN   J1 -> anodo di D1, prima della protezione contro l'inversione
  9V      catodo di D1 -> F2 e F3, il tronco protetto
  9V_BL   F2 -> VIN del buck, il ramo del backlighting

Le etichette locali prendono il prefisso del foglio, quindi le reti si
chiamano /9V_IN, /9V, /9V_BL e il pattern della classe diventa /9V*.

Nessun rame spostato: cambiano solo le stringhe del nome rete su pad e
piste. I gerber escono identici, i nomi non stanno su nessun livello di
fabbricazione.

Netlist verificata: /9V_IN = D1.2 J1.1, /9V = D1.1 F2.2 F3.1,
/9V_BL = C1.1 F2.1 U4.1. ERC identico a prima, DRC 3 violazioni di
libreria, 0 scollegamenti, 0 parita'.

Co-Authored-By: Claude Opus 5 <noreply@anthropic.com>
Connections:
- net Net-(D1-A) renamed /9V_IN
- net Net-(D1-K) renamed /9V
- net Net-(U4-VIN) renamed /9V_BL
Changed lines of the file:
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@@
 			(remove_unused_layers no)
 			(roundrect_rratio 0.15625)
-			(net "Net-(U4-VIN)")
+			(net "/9V_BL")
 			(pintype "passive")
 		)
@@
 			(remove_unused_layers no)
 			(roundrect_rratio 0.078125)
-			(net "Net-(D1-K)")
+			(net "/9V")
 			(pintype "passive")
 		)
@@
 			(layers "*.Cu" "*.Mask")
 			(remove_unused_layers no)
-			(net "Net-(D1-A)")
+			(net "/9V_IN")
 			(pintype "passive")
 		)
@@
 			(layers "*.Cu" "*.Mask")
 			(remove_unused_layers no)
-			(net "Net-(D1-K)")
+			(net "/9V")
 			(pintype "passive")
 		)
@@
 			(layers "F.Cu" "F.Mask" "F.Paste")
 			(roundrect_rratio 0.227273)
-			(net "Net-(U4-VIN)")
+			(net "/9V_BL")
 			(pinfunction "VIN")
 			(pintype "power_in")
@@
 			(remove_unused_layers no)
 			(roundrect_rratio 0.096154)
-			(net "Net-(D1-A)")
+			(net "/9V_IN")
 			(pintype "passive")
 		)
@@
 			(layers "*.Cu" "*.Mask")
 			(remove_unused_layers no)
-			(net "Net-(U4-VIN)")
+			(net "/9V_BL")
 			(pintype "passive")
 		)
@@
 			(layers "*.Cu" "*.Mask")
 			(remove_unused_layers no)
-			(net "Net-(D1-K)")
+			(net "/9V")
 			(pintype "passive")
 		)
@@
 		(width 1)
 		(layer "F.Cu")
-		(net "Net-(U4-VIN)")
+		(net "/9V_BL")
 	)
 	(segment
@@
 		(width 1)
 		(layer "F.Cu")
-		(net "Net-(U4-VIN)")
+		(net "/9V_BL")
 	)
 	(segment
@@
 		(width 1)
 		(layer "F.Cu")
-		(net "Net-(U4-VIN)")
+		(net "/9V_BL")
 	)
 	(segment
@@
 		(width 1)
 		(layer "F.Cu")
-		(net "Net-(D1-K)")
+		(net "/9V")
 	)
 	(segment
@@
 		(width 1)
 		(layer "F.Cu")
-		(net "Net-(D1-K)")
+		(net "/9V")
 	)
 	(segment
@@
 		(width 1)
 		(layer "F.Cu")
-		(net "Net-(D1-K)")
+		(net "/9V")
 	)
 	(segment
@@
 		(width 1)
 		(layer "F.Cu")
-		(net "Net-(D1-K)")
+		(net "/9V")
 	)
 	(segment
@@
 		(width 1)
 		(layer "F.Cu")
-		(net "Net-(D1-K)")
+		(net "/9V")
 	)
 	(segment
@@
 		(width 1)
 		(layer "F.Cu")
-		(net "Net-(D1-K)")
+		(net "/9V")
 	)
 	(segment
@@
 		(width 1)
 		(layer "F.Cu")
-		(net "Net-(D1-K)")
+		(net "/9V")
 	)
 	(segment
@@
 		(width 1)
 		(layer "F.Cu")
-		(net "Net-(D1-K)")
+		(net "/9V")
 	)
 	(segment
@@
 		(width 1)
 		(layer "F.Cu")
-		(net "Net-(D1-K)")
+		(net "/9V")
 	)
 	(segment
@@
 		(width 1)
 		(layer "F.Cu")
-		(net "Net-(D1-A)")
+		(net "/9V_IN")
 	)
 	(segment
@@
 		(width 1)
 		(layer "F.Cu")
-		(net "Net-(D1-A)")
+		(net "/9V_IN")
 	)
 	(segment

Commit message: Drop the PCM symbols the boards did not need
Gli ERC che restavano erano quasi tutti simboli presi da librerie PCM che
bisogna installare a parte. Dove KiCad ha il suo equivalente con gli stessi
pin, tanto vale usarlo e non chiedere niente a chi apre il repository.

PSU: i cinque morsetti passano da PCM_SL_Screw_Terminal a
Connector:Screw_Terminal_01x02. Il simbolo di libreria ha i pin 1.27 mm piu'
in fuori e 1.27 piu' in basso, quindi ogni simbolo e' stato spostato di
altrettanto, ruotato come il componente, e i fili che c'erano restano
attaccati dove stavano. Netlist verificata pin per pin. ERC da 5 a 0.

Cambiare quel simbolo ha pero' rinominato da solo il nodo dei 5 V del
backlighting, che non aveva nome e si chiamava a seconda di quale pin
capitava primo: Net-(LED1-A) e' diventato Net-(J2-Pin_2) e la parita' e'
saltata su dieci pad. Invece di inseguire il nome automatico gliene ho dato
uno vero, 5V_BL, come al ramo dei 9 V.

Dimmer e i due Korry: riallineate alla libreria le definizioni incorporate
di IRLIZ44N e LED. Prima di sostituirle ho confrontato i pin: identici, se
no i fili sarebbero rimasti attaccati al vuoto.

Restano due avvisi, uno sul dimmer e uno sul Korry grande, e li lascio
apposta:
 - il NE555 di Digi-Key ha una disposizione dei pin diversa da quella dei
   555 in libreria, quindi lo scambio vorrebbe rifare tutti i collegamenti;
 - lo switch tattile di Digi-Key numera i pin 1-2 da una parte e 3-4
   dall'altra, Switch:SW_Push_Dual li numera 1-3 e 2-4. Le posizioni
   coincidono, la numerazione no: scambiarlo cambierebbe quali pioli sono
   in corto dentro al pulsante.
Tutti e due i simboli sono incorporati nei file e sono corretti; installare
la libreria Digi-Key li fa tacere.

Stato: sei schede, quattro pulite su tutto. Dimmer 1 ERC e 1 DRC, Korry
grande 1 ERC. Tutte a 0 scollegamenti e 0 parita'.

Co-Authored-By: Claude Opus 5 <noreply@anthropic.com>
Connections:
- net Net-(LED1-A) renamed /5V_BL
Changed lines of the file:
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@@
 			(layers "*.Cu" "*.Mask")
 			(remove_unused_layers no)
-			(net "Net-(LED1-A)")
+			(net "/5V_BL")
 			(pintype "passive")
 		)
@@
 			(layers "*.Cu" "*.Mask")
 			(remove_unused_layers no)
-			(net "Net-(LED1-A)")
+			(net "/5V_BL")
 			(pintype "passive")
 		)
@@
 			(layers "F.Cu" "F.Mask" "F.Paste")
 			(roundrect_rratio 0.2)
-			(net "Net-(LED1-A)")
+			(net "/5V_BL")
 			(pinfunction "A")
 			(pintype "passive")
@@
 			(remove_unused_layers no)
 			(roundrect_rratio 0.15625)
-			(net "Net-(LED1-A)")
+			(net "/5V_BL")
 			(pintype "passive")
 		)
@@
 			(remove_unused_layers no)
 			(roundrect_rratio 0.15625)
-			(net "Net-(LED1-A)")
+			(net "/5V_BL")
 			(pintype "passive")
 		)
@@
 			(layers "F.Cu" "F.Mask" "F.Paste")
 			(roundrect_rratio 0.2)
-			(net "Net-(LED1-A)")
+			(net "/5V_BL")
 			(pinfunction "A")
 			(pintype "passive")
@@
 			(layers "F.Cu" "F.Mask" "F.Paste")
 			(roundrect_rratio 0.227273)
-			(net "Net-(LED1-A)")
+			(net "/5V_BL")
 			(pinfunction "FB")
 			(pintype "input")
@@
 			(layers "*.Cu" "*.Mask")
 			(remove_unused_layers no)
-			(net "Net-(LED1-A)")
+			(net "/5V_BL")
 			(pintype "passive")
 		)
@@
 			(layers "F.Cu" "F.Mask" "F.Paste")
 			(roundrect_rratio 0.2)
-			(net "Net-(LED1-A)")
+			(net "/5V_BL")
 			(pinfunction "A")
 			(pintype "passive")
@@
 			(layers "*.Cu" "*.Mask")
 			(remove_unused_layers no)
-			(net "Net-(LED1-A)")
+			(net "/5V_BL")
 			(pinfunction "2")
 			(pintype "passive")
@@
 		(layer "Edge.Cuts")
 	)
+	(gr_text "5V BACKLIGHT"
+		(at 109.5 24 0)
+		(layer "F.SilkS")
+		(effects
+			(font
+				(size 1 1)
+				(thickness 0.15)
+			)
+		)
+	)
+	(gr_text "5V BACKLIGHT"
+		(at 125 24 0)
+		(layer "F.SilkS")
+		(effects
+			(font
+				(size 1 1)
+				(thickness 0.15)
+			)
+		)
+	)
+	(gr_text "5V BACKLIGHT"
+		(at 140.5 24 0)
+		(layer "F.SilkS")
+		(effects
+			(font
+				(size 1 1)
+				(thickness 0.15)
+			)
+		)
+	)
+	(gr_text "9V IN"
+		(at 140.5 97 0)
+		(layer "F.SilkS")
+		(effects
+			(font
+				(size 1 1)
+				(thickness 0.15)
+			)
+		)
+	)
+	(gr_text "5V MAINBOARD"
+		(at 157.5 25.5 0)
+		(layer "F.SilkS")
+		(effects
+			(font
+				(size 1 1)
+				(thickness 0.15)
+			)
+		)
+	)
 	(gr_text "+"
 		(at 106.65 43.9 0)
@@
 		(width 1)
 		(layer "F.Cu")
-		(net "Net-(LED1-A)")
+		(net "/5V_BL")
 	)
 	(segment
@@
 		(width 1)
 		(layer "F.Cu")
-		(net "Net-(LED1-A)")
+		(net "/5V_BL")
 	)
 	(segment
@@
 		(width 1)
 		(layer "F.Cu")
-		(net "Net-(LED1-A)")
+		(net "/5V_BL")
 	)
 	(segment
@@
 		(width 1)
 		(layer "F.Cu")
-		(net "Net-(LED1-A)")
+		(net "/5V_BL")
 	)
 	(segment
@@
 		(width 1)
 		(layer "F.Cu")
-		(net "Net-(LED1-A)")
+		(net "/5V_BL")
 	)
 	(segment
@@
 		(width 1)
 		(layer "F.Cu")
-		(net "Net-(LED1-A)")
+		(net "/5V_BL")
 	)
 	(segment
@@
 		(width 1)
 		(layer "F.Cu")
-		(net "Net-(LED1-A)")
+		(net "/5V_BL")
 	)
 	(segment
@@
 		(width 1)
 		(layer "F.Cu")
-		(net "Net-(LED1-A)")
+		(net "/5V_BL")
 	)
 	(segment
@@
 		(width 0.5)
 		(layer "F.Cu")
-		(net "Net-(LED1-A)")
+		(net "/5V_BL")
 	)
 	(segment
@@
 		(width 1)
 		(layer "F.Cu")
-		(net "Net-(LED1-A)")
+		(net "/5V_BL")
 	)
 	(segment
@@
 		(width 1)
 		(layer "F.Cu")
-		(net "Net-(LED1-A)")
+		(net "/5V_BL")
 	)
 	(segment
@@
 		(width 0.5)
 		(layer "F.Cu")
-		(net "Net-(LED1-A)")
+		(net "/5V_BL")
 	)
 	(segment
@@
 		(width 1)
 		(layer "F.Cu")
-		(net "Net-(LED1-A)")
+		(net "/5V_BL")
 	)
 	(segment
@@
 		(width 1)
 		(layer "F.Cu")
-		(net "Net-(LED1-A)")
+		(net "/5V_BL")
 	)
 	(segment
@@
 		(width 0.5)
 		(layer "F.Cu")
-		(net "Net-(LED1-A)")
+		(net "/5V_BL")
 	)
 	(segment
@@
 		(width 1)
 		(layer "F.Cu")
-		(net "Net-(LED1-A)")
+		(net "/5V_BL")
 	)
 	(segment
@@
 		(width 1)
 		(layer "F.Cu")
-		(net "Net-(LED1-A)")
+		(net "/5V_BL")
 	)
 	(segment
@@
 		(width 1)
 		(layer "F.Cu")
-		(net "Net-(LED1-A)")
+		(net "/5V_BL")
 	)
 	(segment
@@
 		(width 1)
 		(layer "F.Cu")
-		(net "Net-(LED1-A)")
+		(net "/5V_BL")
 	)
 	(segment
@@
 		(width 1)
 		(layer "F.Cu")
-		(net "Net-(LED1-A)")
+		(net "/5V_BL")
 	)
 	(segment
@@
 		(width 1)
 		(layer "F.Cu")
-		(net "Net-(LED1-A)")
+		(net "/5V_BL")
 	)
 	(segment
@@
 		(width 1)
 		(layer "F.Cu")
-		(net "Net-(LED1-A)")
+		(net "/5V_BL")
 	)
 	(segment
@@
 		(width 0.5)
 		(layer "F.Cu")
-		(net "Net-(LED1-A)")
+		(net "/5V_BL")
 	)
 	(segment
@@
 		(width 1)
 		(layer "F.Cu")
-		(net "Net-(LED1-A)")
+		(net "/5V_BL")
 	)
 	(segment
@@
 		(width 1)
 		(layer "F.Cu")
-		(net "Net-(LED1-A)")
+		(net "/5V_BL")
 	)
 	(segment
@@
 		(width 1)
 		(layer "F.Cu")
-		(net "Net-(LED1-A)")
+		(net "/5V_BL")
 	)
 	(segment
@@
 		(width 0.5)
 		(layer "F.Cu")
-		(net "Net-(LED1-A)")
+		(net "/5V_BL")
 	)
 	(segment
@@
 		(width 1)
 		(layer "F.Cu")
-		(net "Net-(LED1-A)")
+		(net "/5V_BL")
 	)
 	(segment
@@
 		(width 1)
 		(layer "F.Cu")
-		(net "Net-(LED1-A)")
+		(net "/5V_BL")
 	)
 	(segment
@@
 		(width 1)
 		(layer "F.Cu")
-		(net "Net-(LED1-A)")
+		(net "/5V_BL")
 	)
 	(segment
@@
 	)
 	(embedded_fonts no)
-	(gr_text "5V BACKLIGHT"
-		(at 109.5 24 0)
-		(layer "F.SilkS")
-		(effects
-			(font
-				(size 1 1)
-				(thickness 0.15)
-			)
-		)
-	)
-	(gr_text "5V BACKLIGHT"
-		(at 125 24 0)
-		(layer "F.SilkS")
-		(effects
-			(font
-				(size 1 1)
-				(thickness 0.15)
-			)
-		)
-	)
-	(gr_text "5V BACKLIGHT"
-		(at 140.5 24 0)
-		(layer "F.SilkS")
-		(effects
-			(font
-				(size 1 1)
-				(thickness 0.15)
-			)
-		)
-	)
-	(gr_text "5V MAINBOARD"
-		(at 157.5 25.5 0)
-		(layer "F.SilkS")
-		(effects
-			(font
-				(size 1 1)
-				(thickness 0.15)
-			)
-		)
-	)
-	(gr_text "9V IN"
-		(at 140.5 97 0)
-		(layer "F.SilkS")
-		(effects
-			(font
-				(size 1 1)
-				(thickness 0.15)
-			)
-		)
-	)
 )
