File: Korry_Large/KorryLargePCB_SMD.kicad_pcb (KiCad board)
At the start: 2 copper layers, 32.8 x 32 mm, 9 parts, among them J1 BTN+LED, J2 BK_LED

Commit message: Fix the swapped EFIS filenames and rename the backlight nets to +5V
Two naming defects, no electrical change on any board.

EFIS sheets
-----------
The root sheet pointed EFIS_LEFT at efis_right.kicad_sch and EFIS_RIGHT at
efis_left.kicad_sch. The schematic was correct, since the file behind the
LEFT sheet did hold the L_* signals, but the filenames said the opposite and
anyone reading the files from outside KiCad would have been misled.

The two files are swapped and every reference follows: the sheet properties
in the root schematic and the 49 sheetfile entries the footprints carry on
the board. Each file now matches the sheet that loads it.

  netlist   198 nets, 135 components, not one node moved
  ERC       0 violations
  DRC       6 violations, all cosmetic, 0 unconnected, 0 parity issues

Backlight nets
--------------
Every net in the backlighting chain was called +9V while carrying 5 V, on
all four boards. The white LEDs sit behind 91 Ω: at 5 V that is 21 mA, right
at the rating for a 1206 white LED, while 9 V would put them at 65 mA. The
name was a leftover from an earlier design and was the kind of label that
eventually makes someone connect the wrong supply.

Renamed across Korry_Large, Korry_Small, Backlighting_Dimmer and
Backlighting_LEDModule, in both the schematics and the boards: the power
symbol, its value, which is what actually names the net, and the net entries
on the copper. 88 occurrences. None of those boards had a +5V net already,
so nothing was merged.

Verified against the state committed a moment ago: ERC and DRC counts are
identical on all four boards, before and after, and no board gained or lost
a connection.

The Readme drops these two entries and gains the defects that surfaced while
checking: the Backlighting_Dimmer footprints carry their reference in the
value field instead of the schematic value, so a BOM read from that board is
wrong; its terminal block footprint no longer exists in the KiCad library;
four texts on the Korry_Large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
Connections:
- net +9V renamed +5V
Changed lines of the file:
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@@
 	(net 0 "")
 	(net 1 "/LED_INPUT")
-	(net 2 "+9V")
+	(net 2 "+5V")
 	(net 3 "/BTN_INPUT")
 	(net 4 "GND")
@@
 			(layers "*.Cu" "*.Mask")
 			(remove_unused_layers no)
-			(net 2 "+9V")
+			(net 2 "+5V")
 			(pinfunction "Pin_1")
 			(pintype "passive")
@@
 			(layers "B.Cu" "B.Paste" "B.Mask")
 			(roundrect_rratio 0.175439)
-			(net 2 "+9V")
+			(net 2 "+5V")
 			(pinfunction "A")
 			(pintype "passive")

Commit message: Re-annotate the dimmer against its board, set the Korry resistor values
Tidying only. No board changed, no connection moved: all six projects still
report 0 unconnected items and 0 schematic parity issues.

Backlighting_Dimmer was worse than the value mismatch the Readme recorded.
Its schematic and its board disagreed on six reference designators, and
three separate connectors in the schematic all carried J73:

  J73 -> J12, J13, J14     three connectors sharing one reference
  J12 -> J31               J12 was the potentiometer in the schematic and a
                           terminal block on the board
  J93 -> J32
  U2  -> U1

Running Update PCB from Schematic on that board would have pushed those
references onto the copper and left three footprints called J73, against a
silkscreen that is already manufactured. The board is physical reality, so
the schematic was back-annotated from it, values included: R 5K became 5K,
C 470nF became 470nF and so on, which is also the better BOM text.
Schematic parity on that board goes from 6 to 0.

Backlighting_LEDModule had the same problem on one symbol, J73 -> J11.

The Korry resistors had no value in either schematic. Set to the fitted
parts, in the schematics and on the boards: RG 220 ohm for the green
annunciator, RW 91 ohm for the white backlight LED. At 5 V that is about
11 mA and 21 mA.

Three findings are deliberately left as they are, and the Readme now says
why rather than listing them as things to do:

- the dangling terminal block footprint has no replacement in KiCad 10,
  which ships no 2-pin 5.08 mm terminal block. Retargeting it would change
  the pads of a board already made
- the unmirrored + and - markers on the Korry_Large back silkscreen are
  symmetric glyphs, so nothing reads wrong, and mirroring them would move
  them sideways
- the PWR_FLAG the LEDModule wants is a two-click job in Eeschema. That
  file is KiCad 8 and the symbol definition would have to come from a
  KiCad 10 library carrying five toke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
Parts:
- RG-1: value R -> 220
- RW-1: value R -> 91
Changed lines of the file:
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@@
 			)
 		)
-		(property "Value" "R"
+		(property "Value" "220"
 			(at 0 1.82 90)
 			(layer "F.Fab")
@@
 			)
 		)
-		(property "Value" "R"
+		(property "Value" "91"
 			(at 0 1.82 -90)
 			(layer "F.Fab")

Commit message: Align the Korry connector with the mainboard
La mainboard mette GND sul pin 1 di tutti e 34 i suoi connettori a 3 pin. I
Korry avevano pin 1 = pulsante e pin 3 = GND, quindi con un cavetto dritto
la massa finiva sull'ingresso del pulsante e l'ingresso del multiplexer
sulla massa del Korry. Funzionava solo infilando il connettore al
contrario.

Scambiati i pin 1 e 3 sul Korry, che ha un connettore per scheda, e non
sulla mainboard, che ne ha venti e che con GND sul pin 1 e' coerente con se
stessa.

Sullo schema il simbolo di J1 e' specchiato sull'asse X: i pin 1 e 3 si
scambiano di posto e i fili che c'erano finiscono da soli su quello giusto.
Sul rame si sono scambiate le reti dei due pad e si e' rifatta la pista del
pulsante, che ora esce dall'altro capo del connettore; la massa la prende il
piano come prima. Sul Korry grande la pista scansa il pad 3 dello switch,
che e' massa e sta in mezzo.

Scambiate anche le lettere 'G' e 'B' sul serigrafico, che indicano i pin e
sarebbero diventate bugiarde.

Netlist verificata: J1 ora e' 1=GND, 2=LED_INPUT, 3=BTN_INPUT su entrambe.
Le zone sono da riempire.

Co-Authored-By: Claude Opus 5 <noreply@anthropic.com>
Connections:
- J1 pad 1: /BTN_INPUT -> GND
- J1 pad 3: GND -> /BTN_INPUT
Changed lines of the file:
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@@
 			(layers "*.Cu" "*.Mask")
 			(remove_unused_layers no)
-			(net "/BTN_INPUT")
+			(net "GND")
 			(pinfunction "Pin_1")
 			(pintype "passive")
@@
 			(layers "*.Cu" "*.Mask")
 			(remove_unused_layers no)
-			(net "GND")
+			(net "/BTN_INPUT")
 			(pinfunction "Pin_3")
 			(pintype "passive")
@@
 		(layer "User.1")
 	)
-	(gr_text "G"
+	(gr_text "B"
 		(at 58 26.4 0)
 		(layer "F.SilkS")
@@
 		)
 	)
-	(gr_text "B"
+	(gr_text "G"
 		(at 63.3 26.4 0)
 		(layer "F.SilkS")
@@
 	)
 	(segment
-		(start 63.75 23)
-		(end 62.525 24.225)
-		(width 0.25)
-		(layer "F.Cu")
-		(net "/BTN_INPUT")
-	)
-	(segment
-		(start 62.525 34.535)
-		(end 58.01 39.05)
-		(width 0.25)
-		(layer "F.Cu")
-		(net "/BTN_INPUT")
-	)
-	(segment
-		(start 62.525 24.225)
-		(end 62.525 34.535)
-		(width 0.25)
-		(layer "F.Cu")
-		(net "/BTN_INPUT")
-	)
-	(segment
 		(start 67.775 34.1)
 		(end 67.775 32.605)
@@
 	)
 	(embedded_fonts no)
+	(segment
+		(start 58.67 23)
+		(end 58.67 31)
+		(width 0.25)
+		(layer "F.Cu")
+		(net "/BTN_INPUT")
+	)
+	(segment
+		(start 58.67 31)
+		(end 55.8 33.87)
+		(width 0.25)
+		(layer "F.Cu")
+		(net "/BTN_INPUT")
+	)
+	(segment
+		(start 55.8 33.87)
+		(end 55.8 36.84)
+		(width 0.25)
+		(layer "F.Cu")
+		(net "/BTN_INPUT")
+	)
+	(segment
+		(start 55.8 36.84)
+		(end 58.01 39.05)
+		(width 0.25)
+		(layer "F.Cu")
+		(net "/BTN_INPUT")
+	)
 )
