File: Korry_Large/KorryLargePCB_SMD.kicad_pcb (KiCad board)
At the start: 2 copper layers, 32.8 x 32 mm, 9 parts, among them J1 BTN+LED, J2 BK_LED

Commit message: Say on the silkscreen what plugs into each connector
Le schede da fabbricate non si leggevano: quasi tutti i valori stavano su
F.Fab, che non va in stampa, e meta' dei connettori aveva come nome il tipo
di morsetto invece di cosa ci va attaccato.

Nessun valore e' stato riscritto: il nome del componente resta quello che
dice KiCad. Si e' lavorato solo sul serigrafico, in due modi.

I valori che gia' dicono qualcosa di utile sono passati su F.Silk, cosi' si
stampano: Backlighting POT sul dimmer, BTN+LED e BK_LED sui Korry, e i 220 e
91 delle due resistenze, che da montare sono due rettangoli identici.

Dove il valore e' il tipo di morsetto e stampalo non servirebbe a niente, il
valore resta dov'e' e accanto ci va una scritta che dice dove va il filo:

  PSU        J1 -> 9V IN, J2/J3/J4 -> 5V BACKLIGHT, J5 -> 5V MAINBOARD
  Dimmer     J32 -> 5V IN, J12/J13/J14 -> TO LEDMODULE
  LEDModule  J11 -> 5V IN

Ogni posizione e' stata verificata contro pad, altre scritte, contorni
serigrafici e bordo scheda, e poi ricontrollata col DRC, che e' l'unico a
sapere quanto e' larga davvero l'apertura di maschera di un foro di
fissaggio: la scritta di J14 ci finiva sopra, e il valore di J1 sul Korry
grande finiva a cavallo del bordo.

Tutte e cinque le schede: 0 scollegamenti, 0 differenze con lo schema,
nessuna violazione serigrafica. Restano solo gli avvisi di libreria.

Co-Authored-By: Claude Opus 5 <noreply@anthropic.com>
Changed lines of the file:
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@@
 		(property "Value" "220"
 			(at 0 1.82 90)
-			(layer "F.Fab")
+			(layer "F.SilkS")
 			(effects
 				(font
@@
 		(property "Value" "BK_LED"
 			(at 0 4.87 90)
-			(layer "F.Fab")
+			(layer "F.SilkS")
 			(effects
 				(font
@@
 		)
 		(property "Value" "BTN+LED"
-			(at 0 7.41 90)
-			(layer "F.Fab")
+			(at 5.3 2.55 0)
+			(layer "F.SilkS")
 			(effects
 				(font
@@
 		)
 		(property "Value" "91"
-			(at 0 1.82 270)
-			(layer "F.Fab")
-			(effects
-				(font
+			(at -3.33 0 0)
+			(layer "F.SilkS")
+			(effects
+				(font
