File: Mainboard/FCU_Mainboard_v3.kicad_pcb (KiCad board)
At the start: 2 copper layers, 270 x 100 mm, 143 parts, among them J1 R_OLED, J10 AP2, J11 AP1, J12 BootLoader, J13 5V from PSU, J14 ALT_OLED, J15 VSPEED_OLED, J16 R_FD, J17 R_LS, J18 R_CSTR, J19 R_WPT, J2 L_OLED, J20 R_VORD, J21 R_NDB, J22 R_ARPT, J23 LB_PULL, J24 LB_PUSH, J25 LB_hPa/inHg, J26 L_FD, J27 L_LS, J28 L_CSTR, J29 L_WPT, J3 SPD_OLED, J30 SPD/MACH, J31 HDG/TRK, J32 MET_ALT, J33 LVL_OFF, J34 S_PUSH, J35 HDG_ENC, J36 RB_ENC, J37 H_PUSH, J38 RB_PULL, J39 RB_hPa/inHg, J4 HDG_OLED, J40 L_VORD, J41 SPD_ENC, J42 ALT_ENC, J43 A_PUSH, J44 RB_PUSH, J45 A_1H_1K, J46 VS_ENC, J47 L_NDB, J48 VS_PUSH, J49 RVOR/ADF_1, J5 H_T_OLED, J50 RVOR/ADF_2, J51 R_MAP_MODE, J52 L_ARPT, J53 R_MAP_RANGE, J54 L_MAP_MODE, J55 L_MAP_RANGE, J56 LB_ENC, J57 LVOR/ADF_1, J58 LVOR/ADF_2, J6 APPR, J69 S_PULL, J7 EXPED, J70 H_PULL, J71 A_PULL, J72 VS_PULL, J8 LOC, J9 A/THR, P1 USB_B, SW1 SW_DIP_x03, U1 CD74HC4067M, U2 CD74HC4067M, U3 CD74HC4067M, U4 CD74HC4067M, U5 ATMega2560, U6 CH340G, U7 AMS1117-3.3, U8 TPS2115A

Commit message: Name the two autopilot lamp nets after the right autopilot
J10 porta la serigrafia AP2 e aveva sopra AP1_LED con AP2_BTN; J11 porta AP1
e aveva AP2_LED con AP1_BTN. Su un Airbus i due autopiloti sono indipendenti,
quindi ogni connettore deve portare la lampada e il pulsante dello stesso.

Il difetto sta solo nei nomi: le due reti LED arrivano ai pin 96 e 97 del
Mega, adiacenti, e ognuna era gia' cablata al connettore giusto. Scambiare i
due nomi rende coerenti schema, serigrafia e rame senza spostare un
millimetro di pista, e senza toccare la configurazione MobiFlight, che
ragiona per numero di pin.

Ora: J10 (AP2) = AP2_LED + AP2_BTN, J11 (AP1) = AP1_LED + AP1_BTN.
ERC 0, DRC 0, parita' 0.

Co-Authored-By: Claude Opus 5 <noreply@anthropic.com>
Connections:
- J10 pad 2: AP1_LED -> AP2_LED
- J11 pad 2: AP2_LED -> AP1_LED
- U5 pad 96: AP2_LED -> AP1_LED
- U5 pad 97: AP1_LED -> AP2_LED
Routing:
- net AP2_LED: track 59.6 -> 77.7 mm
- net AP1_LED: track 77.7 -> 59.6 mm
Changed lines of the file:
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@@
 			(layers "*.Cu" "*.Mask")
 			(remove_unused_layers no)
-			(net "AP2_LED")
+			(net "AP1_LED")
 			(pinfunction "Pin_2_2")
 			(pintype "passive")
@@
 			(layers "*.Cu" "*.Mask")
 			(remove_unused_layers no)
-			(net "AP1_LED")
+			(net "AP2_LED")
 			(pinfunction "Pin_2_2")
 			(pintype "passive")
@@
 			(size 0.35 1.5)
 			(layers "F.Cu" "F.Mask" "F.Paste")
-			(net "AP2_LED")
+			(net "AP1_LED")
 			(pinfunction "PF1_96")
 			(pintype "bidirectional")
@@
 			(size 0.35 1.5)
 			(layers "F.Cu" "F.Mask" "F.Paste")
-			(net "AP1_LED")
+			(net "AP2_LED")
 			(pinfunction "PF0_97")
 			(pintype "bidirectional")
@@
 		(width 0.2)
 		(layer "F.Cu")
-		(net "AP2_LED")
+		(net "AP1_LED")
 	)
 	(segment
@@
 		(width 0.2)
 		(layer "F.Cu")
-		(net "AP2_LED")
+		(net "AP1_LED")
 	)
 	(segment
@@
 		(width 0.2)
 		(layer "F.Cu")
-		(net "AP2_LED")
+		(net "AP1_LED")
 	)
 	(segment
@@
 		(width 0.2)
 		(layer "F.Cu")
-		(net "AP2_LED")
+		(net "AP1_LED")
 	)
 	(via
@@
 		)
 		(filling no)
-		(net "AP2_LED")
+		(net "AP1_LED")
 	)
 	(segment
@@
 		(width 0.2)
 		(layer "B.Cu")
-		(net "AP2_LED")
+		(net "AP1_LED")
 	)
 	(segment
@@
 		(width 0.2)
 		(layer "B.Cu")
-		(net "AP2_LED")
+		(net "AP1_LED")
 	)
 	(segment
@@
 		(width 0.2)
 		(layer "B.Cu")
-		(net "AP2_LED")
+		(net "AP1_LED")
 	)
 	(segment
@@
 		(width 0.2)
 		(layer "B.Cu")
-		(net "AP2_LED")
+		(net "AP1_LED")
 	)
 	(segment
@@
 		(width 0.2)
 		(layer "B.Cu")
-		(net "AP2_LED")
+		(net "AP1_LED")
 	)
 	(segment
@@
 		(width 0.2)
 		(layer "B.Cu")
-		(net "AP2_LED")
+		(net "AP1_LED")
 	)
 	(segment
@@
 		(width 0.2)
 		(layer "B.Cu")
-		(net "AP2_LED")
+		(net "AP1_LED")
 	)
 	(segment
@@
 		(width 0.2)
 		(layer "F.Cu")
-		(net "AP1_LED")
+		(net "AP2_LED")
 	)
 	(segment
@@
 		(width 0.2)
 		(layer "F.Cu")
-		(net "AP1_LED")
+		(net "AP2_LED")
 	)
 	(segment
@@
 		(width 0.2)
 		(layer "F.Cu")
-		(net "AP1_LED")
+		(net "AP2_LED")
 	)
 	(via
@@
 		)
 		(filling no)
-		(net "AP1_LED")
+		(net "AP2_LED")
 	)
 	(segment
@@
 		(width 0.2)
 		(layer "B.Cu")
-		(net "AP1_LED")
+		(net "AP2_LED")
 	)
 	(segment
@@
 		(width 0.2)
 		(layer "B.Cu")
-		(net "AP1_LED")
+		(net "AP2_LED")
 	)
 	(segment
@@
 		(width 0.2)
 		(layer "B.Cu")
-		(net "AP1_LED")
+		(net "AP2_LED")
 	)
 	(segment
@@
 		(width 0.2)
 		(layer "B.Cu")
-		(net "AP1_LED")
+		(net "AP2_LED")
 	)
 	(segment
@@
 		(width 0.2)
 		(layer "B.Cu")
-		(net "AP1_LED")
+		(net "AP2_LED")
 	)
 	(segment
@@
 		(width 0.2)
 		(layer "B.Cu")
-		(net "AP1_LED")
+		(net "AP2_LED")
 	)
 	(segment
@@
 		(width 0.2)
 		(layer "B.Cu")
-		(net "AP1_LED")
+		(net "AP2_LED")
 	)
 	(segment
@@
 		(width 0.2)
 		(layer "B.Cu")
-		(net "AP1_LED")
+		(net "AP2_LED")
 	)
 	(segment
@@
 		(width 0.2)
 		(layer "B.Cu")
-		(net "AP1_LED")
+		(net "AP2_LED")
 	)
 	(segment
@@
 		(width 0.2)
 		(layer "B.Cu")
-		(net "AP1_LED")
+		(net "AP2_LED")
 	)
 	(segment
@@
 		(width 0.2)
 		(layer "B.Cu")
-		(net "AP1_LED")
+		(net "AP2_LED")
 	)
 	(segment
@@
 		(width 0.2)
 		(layer "B.Cu")
-		(net "AP1_LED")
+		(net "AP2_LED")
 	)
 	(segment

Commit message: Label the two screws of the mainboard power terminal
La mainboard era gia' etichettata bene: su 196 pad di connettore, 194
avevano la loro scritta accanto, GND / LED / BTN sui venti che vanno ai
Korry, L e R sugli encoder, VOR e ADF sui selettori, hPa e inHg sui baro.

Gli unici due scoperti erano quelli di J13, cioe' il morsetto aggiunto in
questa sessione per i 5 V dalla PSU: il nome del connettore si leggeva ma
non quale vite fosse la massa. Ora c'e' GND sul pin 1 e 5V sul pin 2.

DRC: 0 violazioni, 0 scollegamenti, 0 parita'.

Co-Authored-By: Claude Opus 5 <noreply@anthropic.com>
Other:
- board text added: "5V"
Changed lines of the file:
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@@
 	)
 	(embedded_fonts no)
+	(gr_text "GND"
+		(at 271.9 40 0)
+		(layer "F.SilkS")
+		(effects
+			(font
+				(size 1 1)
+				(thickness 0.15)
+			)
+		)
+	)
+	(gr_text "5V"
+		(at 271.9 35 0)
+		(layer "F.SilkS")
+		(effects
+			(font
+				(size 1 1)
+				(thickness 0.15)
+			)
+		)
+	)
 )
