File: Backlighting_Dimmer/Backlighting_PCB.kicad_pcb (KiCad board)
At the start: 2 copper layers, 43.2 x 55 mm, 19 parts, among them J12 BOARD_CONN, J13 BOARD_CONN, J14 BOARD_CONN, J31 Backlighting POT, J32 Screw_Terminal_01x02, Q1 IRLIZ44N, U1 NE555P

Commit message: Fix the swapped EFIS filenames and rename the backlight nets to +5V
Two naming defects, no electrical change on any board.

EFIS sheets
-----------
The root sheet pointed EFIS_LEFT at efis_right.kicad_sch and EFIS_RIGHT at
efis_left.kicad_sch. The schematic was correct, since the file behind the
LEFT sheet did hold the L_* signals, but the filenames said the opposite and
anyone reading the files from outside KiCad would have been misled.

The two files are swapped and every reference follows: the sheet properties
in the root schematic and the 49 sheetfile entries the footprints carry on
the board. Each file now matches the sheet that loads it.

  netlist   198 nets, 135 components, not one node moved
  ERC       0 violations
  DRC       6 violations, all cosmetic, 0 unconnected, 0 parity issues

Backlight nets
--------------
Every net in the backlighting chain was called +9V while carrying 5 V, on
all four boards. The white LEDs sit behind 91 Ω: at 5 V that is 21 mA, right
at the rating for a 1206 white LED, while 9 V would put them at 65 mA. The
name was a leftover from an earlier design and was the kind of label that
eventually makes someone connect the wrong supply.

Renamed across Korry_Large, Korry_Small, Backlighting_Dimmer and
Backlighting_LEDModule, in both the schematics and the boards: the power
symbol, its value, which is what actually names the net, and the net entries
on the copper. 88 occurrences. None of those boards had a +5V net already,
so nothing was merged.

Verified against the state committed a moment ago: ERC and DRC counts are
identical on all four boards, before and after, and no board gained or lost
a connection.

The Readme drops these two entries and gains the defects that surfaced while
checking: the Backlighting_Dimmer footprints carry their reference in the
value field instead of the schematic value, so a BOM read from that board is
wrong; its terminal block footprint no longer exists in the KiCad library;
four texts on the Korry_Large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
Connections:
- net +9V renamed +5V
Changed lines of the file:
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@@
 	(net 5 "Net-(D1-A)")
 	(net 6 "Net-(D2-A)")
-	(net 7 "+9V")
+	(net 7 "+5V")
 	(net 8 "Net-(Q1-G)")
 	(net 9 "Net-(J12-Pin_2)")
@@
 			(layers "*.Cu" "*.Mask")
 			(remove_unused_layers no)
-			(net 7 "+9V")
+			(net 7 "+5V")
 			(pintype "passive")
 		)
@@
 			(layers "*.Cu" "*.Mask")
 			(remove_unused_layers no)
-			(net 7 "+9V")
+			(net 7 "+5V")
 			(pinfunction "Pin_1")
 			(pintype "passive")
@@
 			(layers "*.Cu" "*.Mask")
 			(remove_unused_layers no)
-			(net 7 "+9V")
+			(net 7 "+5V")
 			(pintype "passive")
 		)
@@
 			(layers "*.Cu" "*.Mask")
 			(remove_unused_layers no)
-			(net 7 "+9V")
+			(net 7 "+5V")
 			(pintype "passive")
 		)
@@
 			(layers "*.Cu" "*.Mask")
 			(remove_unused_layers no)
-			(net 7 "+9V")
+			(net 7 "+5V")
 			(pinfunction "Pin_1")
 			(pintype "passive")
@@
 			(layers "*.Cu" "*.Mask")
 			(remove_unused_layers no)
-			(net 7 "+9V")
+			(net 7 "+5V")
 			(pinfunction "Pin_1")
 			(pintype "passive")
@@
 			(layers "*.Cu" "*.Mask")
 			(remove_unused_layers no)
-			(net 7 "+9V")
+			(net 7 "+5V")
 			(pinfunction "RESET")
 			(pintype "input")
@@
 			(layers "*.Cu" "*.Mask")
 			(remove_unused_layers no)
-			(net 7 "+9V")
+			(net 7 "+5V")
 			(pinfunction "VCC")
 			(pintype "power_in")
@@
 			(layers "*.Cu" "*.Mask")
 			(remove_unused_layers no)
-			(net 7 "+9V")
+			(net 7 "+5V")
 			(pinfunction "Pin_1")
 			(pintype "passive")

Commit message: Say on the silkscreen what plugs into each connector
Le schede da fabbricate non si leggevano: quasi tutti i valori stavano su
F.Fab, che non va in stampa, e meta' dei connettori aveva come nome il tipo
di morsetto invece di cosa ci va attaccato.

Nessun valore e' stato riscritto: il nome del componente resta quello che
dice KiCad. Si e' lavorato solo sul serigrafico, in due modi.

I valori che gia' dicono qualcosa di utile sono passati su F.Silk, cosi' si
stampano: Backlighting POT sul dimmer, BTN+LED e BK_LED sui Korry, e i 220 e
91 delle due resistenze, che da montare sono due rettangoli identici.

Dove il valore e' il tipo di morsetto e stampalo non servirebbe a niente, il
valore resta dov'e' e accanto ci va una scritta che dice dove va il filo:

  PSU        J1 -> 9V IN, J2/J3/J4 -> 5V BACKLIGHT, J5 -> 5V MAINBOARD
  Dimmer     J32 -> 5V IN, J12/J13/J14 -> TO LEDMODULE
  LEDModule  J11 -> 5V IN

Ogni posizione e' stata verificata contro pad, altre scritte, contorni
serigrafici e bordo scheda, e poi ricontrollata col DRC, che e' l'unico a
sapere quanto e' larga davvero l'apertura di maschera di un foro di
fissaggio: la scritta di J14 ci finiva sopra, e il valore di J1 sul Korry
grande finiva a cavallo del bordo.

Tutte e cinque le schede: 0 scollegamenti, 0 differenze con lo schema,
nessuna violazione serigrafica. Restano solo gli avvisi di libreria.

Co-Authored-By: Claude Opus 5 <noreply@anthropic.com>
Other:
- board text added: "5V IN"
- board text added: "TO LEDMODULE"
Changed lines of the file:
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@@
 		)
 		(property "Value" "Backlighting POT"
-			(at 0 7.41 0)
-			(layer "F.Fab")
+			(at -4.07 7.41 0)
+			(layer "F.SilkS")
 			(effects
 				(font
@@
 	)
 	(embedded_fonts no)
+	(gr_text "5V IN"
+		(at 79.2 36 0)
+		(layer "F.SilkS")
+		(effects
+			(font
+				(size 1 1)
+				(thickness 0.15)
+			)
+		)
+	)
+	(gr_text "TO LEDMODULE"
+		(at 63.94 72.4 0)
+		(layer "F.SilkS")
+		(effects
+			(font
+				(size 1 1)
+				(thickness 0.15)
+			)
+		)
+	)
+	(gr_text "TO LEDMODULE"
+		(at 79.1 72.4 0)
+		(layer "F.SilkS")
+		(effects
+			(font
+				(size 1 1)
+				(thickness 0.15)
+			)
+		)
+	)
+	(gr_text "TO LEDMODULE"
+		(at 94.22 72.4 0)
+		(layer "F.SilkS")
+		(effects
+			(font
+				(size 1 1)
+				(thickness 0.15)
+			)
+		)
+	)
 )

Commit message: Use the same terminal block everywhere
Le due schede backlighting stavano su TerminalBlock_bornier-2_P5.08mm, che
la libreria KiCad 10 non ha piu'. Il morsetto e' lo stesso che sta su PSU e
mainboard, quindi ora lo e' anche nei file: Phoenix PT-1,5-2-5.0-H, su
J12, J13, J14 e J32 del dimmer e su J11 del LEDModule.

Cosa cambia nel rame: passo 5.08 -> 5.00, pad 3.0 -> 2.6, foro 1.52 -> 1.30.
Gli 8 centesimi di passo non li sente nessuno; il foro piu' stretto e' la
misura giusta per quel morsetto.

Il corpo Phoenix e' pero' 1.64 mm piu' profondo del bornier, e questo si
sente:
 - J12, J13 e J14 arrivavano a 0.04 mm dal courtyard dei fori di fissaggio.
   Alzati di un decimo;
 - J32 e J11 stavano a filo del bordo scheda col vecchio corpo e col nuovo
   sporgevano. Rientrati, J11 esattamente dove stava prima la sua faccia
   esterna;
 - le estremita' delle piste sono state riagganciate ai nuovi centri dei
   pad, 13 in tutto, invece di lasciarle fuori centro;
 - le tre scritte TO LEDMODULE non ci stavano piu' sopra ai morsetti: una
   sola sotto alla fila, che sono tre uscite identiche.

Resta un solo avviso sul dimmer, ed e' geometria, non una svista: il
disegno dell'imbocco filo di J32 sfiora il bordo scheda a 0.02 mm. Per
rientrare J32 dovrebbe scendere, ma sotto ha C4 a 0.04 mm dal suo
courtyard: la finestra utile e' alta 10.49 mm per un corpo da 10. Tenuto
l'errore di courtyard risolto e lasciato l'avviso serigrafico, che vuol dire
solo che un pezzetto di inchiostro viene tagliato al bordo.

I problemi noti sono ora vuoti. Le zone delle due schede sono da riempire.

Co-Authored-By: Claude Opus 5 <noreply@anthropic.com>
Parts:
- J12, J13, J14, J32: footprint TerminalBlock:TerminalBlock_bornier-2_P5.08mm -> TerminalBlock_Phoenix:TerminalBlock_Phoenix_PT-1,5-2-5.0-H_1x02_P5.00mm_Horizontal
- moved J32 1.50 mm to (81.8, 30.8)
- moved J12 0.10 mm to (61.4, 67.6)
- moved J13 0.10 mm to (76.6, 67.7)
- moved J14 0.10 mm to (91.7, 67.6)
