File: Backlighting_Dimmer/Backlighting_PCB.kicad_sch (KiCad schematic)
At the start: 19 parts, among them J12 Backlighting POT, J73 BOARD_CONN, J93 Screw_Terminal_01x02, Q1 IRLIZ44N, U2 NE555P

Commit message: Fix the swapped EFIS filenames and rename the backlight nets to +5V
Two naming defects, no electrical change on any board.

EFIS sheets
-----------
The root sheet pointed EFIS_LEFT at efis_right.kicad_sch and EFIS_RIGHT at
efis_left.kicad_sch. The schematic was correct, since the file behind the
LEFT sheet did hold the L_* signals, but the filenames said the opposite and
anyone reading the files from outside KiCad would have been misled.

The two files are swapped and every reference follows: the sheet properties
in the root schematic and the 49 sheetfile entries the footprints carry on
the board. Each file now matches the sheet that loads it.

  netlist   198 nets, 135 components, not one node moved
  ERC       0 violations
  DRC       6 violations, all cosmetic, 0 unconnected, 0 parity issues

Backlight nets
--------------
Every net in the backlighting chain was called +9V while carrying 5 V, on
all four boards. The white LEDs sit behind 91 Ω: at 5 V that is 21 mA, right
at the rating for a 1206 white LED, while 9 V would put them at 65 mA. The
name was a leftover from an earlier design and was the kind of label that
eventually makes someone connect the wrong supply.

Renamed across Korry_Large, Korry_Small, Backlighting_Dimmer and
Backlighting_LEDModule, in both the schematics and the boards: the power
symbol, its value, which is what actually names the net, and the net entries
on the copper. 88 occurrences. None of those boards had a +5V net already,
so nothing was merged.

Verified against the state committed a moment ago: ERC and DRC counts are
identical on all four boards, before and after, and no board gained or lost
a connection.

The Readme drops these two entries and gains the defects that surfaced while
checking: the Backlighting_Dimmer footprints carry their reference in the
value field instead of the schematic value, so a BOM read from that board is
wrong; its terminal block footprint no longer exists in the KiCad library;
four texts on the Korry_Large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
Connections:
- net +9V renamed +5V
Changed lines of the file:
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@@
 	)
 	(symbol
-		(lib_id "power:+9V")
+		(lib_id "power:+5V")
 		(at 233.68 46.99 0)
 		(unit 1)
@@
 			)
 		)
-		(property "Value" "+9V"
+		(property "Value" "+5V"
 			(at 233.68 41.91 0)
 			(effects
@@
 	)
 	(symbol
-		(lib_id "power:+9V")
+		(lib_id "power:+5V")
 		(at 133.35 153.67 270)
 		(unit 1)
@@
 			)
 		)
-		(property "Value" "+9V"
+		(property "Value" "+5V"
 			(at 137.16 153.67 90)
 			(effects
@@
 	)
 	(symbol
-		(lib_id "power:+9V")
+		(lib_id "power:+5V")
 		(at 154.94 45.72 0)
 		(unit 1)
@@
 			)
 		)
-		(property "Value" "+9V"
+		(property "Value" "+5V"
 			(at 154.94 40.64 0)
 			(effects
@@
 	)
 	(symbol
-		(lib_id "power:+9V")
+		(lib_id "power:+5V")
 		(at 255.27 46.99 0)
 		(unit 1)
@@
 			)
 		)
-		(property "Value" "+9V"
+		(property "Value" "+5V"
 			(at 255.27 41.91 0)
 			(effects
@@
 	)
 	(symbol
-		(lib_id "power:+9V")
+		(lib_id "power:+5V")
 		(at 210.82 46.99 0)
 		(unit 1)
@@
 			)
 		)
-		(property "Value" "+9V"
+		(property "Value" "+5V"
 			(at 210.82 41.91 0)
 			(effects
@@
 	)
 	(symbol
-		(lib_id "power:+9V")
+		(lib_id "power:+5V")
 		(at 190.5 57.15 0)
 		(unit 1)
@@
 			)
 		)
-		(property "Value" "+9V"
+		(property "Value" "+5V"
 			(at 190.5 52.07 0)
 			(effects

Commit message: Re-annotate the dimmer against its board, set the Korry resistor values
Tidying only. No board changed, no connection moved: all six projects still
report 0 unconnected items and 0 schematic parity issues.

Backlighting_Dimmer was worse than the value mismatch the Readme recorded.
Its schematic and its board disagreed on six reference designators, and
three separate connectors in the schematic all carried J73:

  J73 -> J12, J13, J14     three connectors sharing one reference
  J12 -> J31               J12 was the potentiometer in the schematic and a
                           terminal block on the board
  J93 -> J32
  U2  -> U1

Running Update PCB from Schematic on that board would have pushed those
references onto the copper and left three footprints called J73, against a
silkscreen that is already manufactured. The board is physical reality, so
the schematic was back-annotated from it, values included: R 5K became 5K,
C 470nF became 470nF and so on, which is also the better BOM text.
Schematic parity on that board goes from 6 to 0.

Backlighting_LEDModule had the same problem on one symbol, J73 -> J11.

The Korry resistors had no value in either schematic. Set to the fitted
parts, in the schematics and on the boards: RG 220 ohm for the green
annunciator, RW 91 ohm for the white backlight LED. At 5 V that is about
11 mA and 21 mA.

Three findings are deliberately left as they are, and the Readme now says
why rather than listing them as things to do:

- the dangling terminal block footprint has no replacement in KiCad 10,
  which ships no 2-pin 5.08 mm terminal block. Retargeting it would change
  the pads of a board already made
- the unmirrored + and - markers on the Korry_Large back silkscreen are
  symmetric glyphs, so nothing reads wrong, and mirroring them would move
  them sideways
- the PWR_FLAG the LEDModule wants is a two-click job in Eeschema. That
  file is KiCad 8 and the symbol definition would have to come from a
  KiCad 10 library carrying five toke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
Parts:
- C1: value C 470nF -> 470nF
- C2: value C 10nF -> 10nF
- C3: value C 100nF -> 100nF
- C4: value C 10uF -> 10uF
- R1: value R 1K -> 1K
- R2: value R 5K -> 5K
- renumbered J73 to J12, J73 to J13, J73 to J14, J12 to J31, J93 to J32, U2 to U1
Changed lines of the file:
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@@
 		(dnp no)
 		(fields_autoplaced yes)
-		(property "Reference" "J73"
+		(property "Reference" "J14"
 			(at 218.44 54.61 0)
 			(effects
@@
 			(project "FCU_Mainboard_v2"
 				(path "/3267b3f3-6c63-480a-8354-1757ed0a4fd3/7ac51fd7-f93f-468f-8c10-b814dd9f4aef"
-					(reference "J73")
+					(reference "J14")
 					(unit 1)
 				)
@@
 			)
 		)
-		(property "Value" "R 5K"
+		(property "Value" "5K"
 			(at 224.79 104.14 0)
 			(effects
@@
 			)
 		)
-		(property "Value" "C 10nF"
+		(property "Value" "10nF"
 			(at 181.61 111.76 0)
 			(effects
@@
 		(dnp no)
 		(fields_autoplaced yes)
-		(property "Reference" "J93"
+		(property "Reference" "J32"
 			(at 144.78 165.1 0)
 			(effects
@@
 			(project "FCU_Mainboard_v2"
 				(path "/3267b3f3-6c63-480a-8354-1757ed0a4fd3/7ac51fd7-f93f-468f-8c10-b814dd9f4aef"
-					(reference "J93")
+					(reference "J32")
 					(unit 1)
 				)
@@
 			)
 		)
-		(property "Value" "C 10uF"
+		(property "Value" "10uF"
 			(at 199.39 82.55 90)
 			(effects
@@
 			)
 		)
-		(property "Value" "R 1K"
+		(property "Value" "1K"
 			(at 157.48 54.61 0)
 			(effects
@@
 		(dnp no)
 		(fields_autoplaced yes)
-		(property "Reference" "U2"
+		(property "Reference" "U1"
 			(at 192.6941 83.82 0)
 			(effects
@@
 			(project "FCU_Mainboard_v2"
 				(path "/3267b3f3-6c63-480a-8354-1757ed0a4fd3/7ac51fd7-f93f-468f-8c10-b814dd9f4aef"
-					(reference "U2")
+					(reference "U1")
 					(unit 1)
 				)
@@
 			)
 		)
-		(property "Value" "C 100nF"
+		(property "Value" "100nF"
 			(at 196.85 66.04 90)
 			(effects
@@
 		(dnp no)
 		(fields_autoplaced yes)
-		(property "Reference" "J73"
+		(property "Reference" "J13"
 			(at 241.3 54.61 0)
 			(effects
@@
 			(project "FCU_Mainboard_v2"
 				(path "/3267b3f3-6c63-480a-8354-1757ed0a4fd3/7ac51fd7-f93f-468f-8c10-b814dd9f4aef"
-					(reference "J73")
+					(reference "J13")
 					(unit 1)
 				)
@@
 		(dnp no)
 		(fields_autoplaced yes)
-		(property "Reference" "J73"
+		(property "Reference" "J12"
 			(at 262.89 54.61 0)
 			(effects
@@
 			(project "FCU_Mainboard_v2"
 				(path "/3267b3f3-6c63-480a-8354-1757ed0a4fd3/7ac51fd7-f93f-468f-8c10-b814dd9f4aef"
-					(reference "J73")
+					(reference "J12")
 					(unit 1)
 				)
@@
 			)
 		)
-		(property "Value" "C 470nF"
+		(property "Value" "470nF"
 			(at 158.75 109.22 0)
 			(effects
@@
 		(on_board yes)
 		(dnp no)
-		(property "Reference" "J12"
+		(property "Reference" "J31"
 			(at 149.86 83.82 90)
 			(effects
@@
 			(project "FCU_Mainboard_v2"
 				(path "/3267b3f3-6c63-480a-8354-1757ed0a4fd3"
-					(reference "J12")
-					(unit 1)
-				)
+					(reference "J31")
+					(unit 1)
+				)

Commit message: Use the same terminal block everywhere
Le due schede backlighting stavano su TerminalBlock_bornier-2_P5.08mm, che
la libreria KiCad 10 non ha piu'. Il morsetto e' lo stesso che sta su PSU e
mainboard, quindi ora lo e' anche nei file: Phoenix PT-1,5-2-5.0-H, su
J12, J13, J14 e J32 del dimmer e su J11 del LEDModule.

Cosa cambia nel rame: passo 5.08 -> 5.00, pad 3.0 -> 2.6, foro 1.52 -> 1.30.
Gli 8 centesimi di passo non li sente nessuno; il foro piu' stretto e' la
misura giusta per quel morsetto.

Il corpo Phoenix e' pero' 1.64 mm piu' profondo del bornier, e questo si
sente:
 - J12, J13 e J14 arrivavano a 0.04 mm dal courtyard dei fori di fissaggio.
   Alzati di un decimo;
 - J32 e J11 stavano a filo del bordo scheda col vecchio corpo e col nuovo
   sporgevano. Rientrati, J11 esattamente dove stava prima la sua faccia
   esterna;
 - le estremita' delle piste sono state riagganciate ai nuovi centri dei
   pad, 13 in tutto, invece di lasciarle fuori centro;
 - le tre scritte TO LEDMODULE non ci stavano piu' sopra ai morsetti: una
   sola sotto alla fila, che sono tre uscite identiche.

Resta un solo avviso sul dimmer, ed e' geometria, non una svista: il
disegno dell'imbocco filo di J32 sfiora il bordo scheda a 0.02 mm. Per
rientrare J32 dovrebbe scendere, ma sotto ha C4 a 0.04 mm dal suo
courtyard: la finestra utile e' alta 10.49 mm per un corpo da 10. Tenuto
l'errore di courtyard risolto e lasciato l'avviso serigrafico, che vuol dire
solo che un pezzetto di inchiostro viene tagliato al bordo.

I problemi noti sono ora vuoti. Le zone delle due schede sono da riempire.

Co-Authored-By: Claude Opus 5 <noreply@anthropic.com>
Parts:
- J12, J13, J14, J32: footprint TerminalBlock:TerminalBlock_bornier-2_P5.08mm -> TerminalBlock_Phoenix:TerminalBlock_Phoenix_PT-1,5-2-5.0-H_1x02_P5.00mm_Horizontal
Changed lines of the file:
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@@
 			)
 		)
-		(property "Footprint" "TerminalBlock:TerminalBlock_bornier-2_P5.08mm"
+		(property "Footprint" "TerminalBlock_Phoenix:TerminalBlock_Phoenix_PT-1,5-2-5.0-H_1x02_P5.00mm_Horizontal"
 			(at 215.9 54.61 0)
 			(hide yes)
@@
 			)
 		)
-		(property "Footprint" "TerminalBlock:TerminalBlock_bornier-2_P5.08mm"
+		(property "Footprint" "TerminalBlock_Phoenix:TerminalBlock_Phoenix_PT-1,5-2-5.0-H_1x02_P5.00mm_Horizontal"
 			(at 142.24 165.1 0)
 			(hide yes)
@@
 			)
 		)
-		(property "Footprint" "TerminalBlock:TerminalBlock_bornier-2_P5.08mm"
+		(property "Footprint" "TerminalBlock_Phoenix:TerminalBlock_Phoenix_PT-1,5-2-5.0-H_1x02_P5.00mm_Horizontal"
 			(at 238.76 54.61 0)
 			(hide yes)
@@
 			)
 		)
-		(property "Footprint" "TerminalBlock:TerminalBlock_bornier-2_P5.08mm"
+		(property "Footprint" "TerminalBlock_Phoenix:TerminalBlock_Phoenix_PT-1,5-2-5.0-H_1x02_P5.00mm_Horizontal"
 			(at 260.35 54.61 0)
 			(hide yes)

Commit message: Keep the last two Digi-Key symbols in the repository
L'ERC segnalava due simboli presi dalla libreria Digi-Key, che non sta nel
Plugin and Content Manager e si scarica a mano da GitHub, per giunta ancora
nel formato .lib di KiCad 5. Per due simboli non vale la pena.

Erano gia' incorporati negli schemi e corretti: mancava solo una libreria a
cui attribuirli. Estratti in due file accanto ai rispettivi progetti, con la
loro sym-lib-table, come si era gia' fatto per il TPS2115A sulla mainboard:

  Backlighting_Dimmer/NE555P.kicad_sym
  Korry_Large/1825910-6.kicad_sym

Sono i simboli con cui le schede sono state disegnate, non equivalenti di
libreria, il che conta soprattutto per il pulsante: Switch:SW_Push_Dual mette
i pin nelle stesse identiche posizioni ma li numera 1-3 e 2-4 dove questo li
numera 1-2 e 3-4, quindi sostituirlo cambierebbe quali pioli sono in corto
dentro al pulsante.

Verificato che i due file sono leggibili da KiCad e che le netlist non si
muovono: NE555 con gli otto pin sulle stesse reti, e sul pulsante pin 1 su
BTN_INPUT, pin 3 su massa, 2 e 4 scollegati come prima.

Sei schede, ERC pulito su tutte. DRC pulito su cinque, piu' l'avviso
serigrafico di J32 sul dimmer. 0 scollegamenti e 0 parita' ovunque.
Delle librerie da installare ne resta una sola, la Alternate KiCad, e serve
per i footprint dei LED e degli Schottky.

Co-Authored-By: Claude Opus 5 <noreply@anthropic.com>
Parts:
- U1: symbol dk_Clock-Timing-Programmable-Timers-and-Oscillators:NE555P -> NE555P:NE555P
Changed lines of the file:
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@@
 	)
 	(symbol
-		(lib_id "dk_Clock-Timing-Programmable-Timers-and-Oscillators:NE555P")
+		(lib_id "NE555P:NE555P")
 		(at 190.5 93.98 0)
 		(unit 1)
