File: Backlighting_LEDModule/Backlighting_LEDModule_PCB.kicad_sch (KiCad schematic)
At the start: 6 parts, among them J1 Conn_02x10_Odd_Even, J2 Conn_02x10_Odd_Even, J73 BOARD_CONN

Commit message: Fix the swapped EFIS filenames and rename the backlight nets to +5V
Two naming defects, no electrical change on any board.

EFIS sheets
-----------
The root sheet pointed EFIS_LEFT at efis_right.kicad_sch and EFIS_RIGHT at
efis_left.kicad_sch. The schematic was correct, since the file behind the
LEFT sheet did hold the L_* signals, but the filenames said the opposite and
anyone reading the files from outside KiCad would have been misled.

The two files are swapped and every reference follows: the sheet properties
in the root schematic and the 49 sheetfile entries the footprints carry on
the board. Each file now matches the sheet that loads it.

  netlist   198 nets, 135 components, not one node moved
  ERC       0 violations
  DRC       6 violations, all cosmetic, 0 unconnected, 0 parity issues

Backlight nets
--------------
Every net in the backlighting chain was called +9V while carrying 5 V, on
all four boards. The white LEDs sit behind 91 Ω: at 5 V that is 21 mA, right
at the rating for a 1206 white LED, while 9 V would put them at 65 mA. The
name was a leftover from an earlier design and was the kind of label that
eventually makes someone connect the wrong supply.

Renamed across Korry_Large, Korry_Small, Backlighting_Dimmer and
Backlighting_LEDModule, in both the schematics and the boards: the power
symbol, its value, which is what actually names the net, and the net entries
on the copper. 88 occurrences. None of those boards had a +5V net already,
so nothing was merged.

Verified against the state committed a moment ago: ERC and DRC counts are
identical on all four boards, before and after, and no board gained or lost
a connection.

The Readme drops these two entries and gains the defects that surfaced while
checking: the Backlighting_Dimmer footprints carry their reference in the
value field instead of the schematic value, so a BOM read from that board is
wrong; its terminal block footprint no longer exists in the KiCad library;
four texts on the Korry_Large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
Connections:
- net +9V renamed +5V
Changed lines of the file:
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@@
 	)
 	(symbol
-		(lib_id "power:+9V")
+		(lib_id "power:+5V")
 		(at 77.47 124.46 180)
 		(unit 1)
@@
 			)
 		)
-		(property "Value" "+9V"
+		(property "Value" "+5V"
 			(at 77.47 131.572 90)
 			(effects
@@
 	)
 	(symbol
-		(lib_id "power:+9V")
+		(lib_id "power:+5V")
 		(at 46.99 124.46 180)
 		(unit 1)
@@
 			)
 		)
-		(property "Value" "+9V"
+		(property "Value" "+5V"
 			(at 46.99 131.572 90)
 			(effects
@@
 	)
 	(symbol
-		(lib_id "power:+9V")
+		(lib_id "power:+5V")
 		(at 62.23 143.51 90)
 		(unit 1)
@@
 			)
 		)
-		(property "Value" "+9V"
+		(property "Value" "+5V"
 			(at 55.118 143.51 90)
 			(effects

Commit message: Re-annotate the dimmer against its board, set the Korry resistor values
Tidying only. No board changed, no connection moved: all six projects still
report 0 unconnected items and 0 schematic parity issues.

Backlighting_Dimmer was worse than the value mismatch the Readme recorded.
Its schematic and its board disagreed on six reference designators, and
three separate connectors in the schematic all carried J73:

  J73 -> J12, J13, J14     three connectors sharing one reference
  J12 -> J31               J12 was the potentiometer in the schematic and a
                           terminal block on the board
  J93 -> J32
  U2  -> U1

Running Update PCB from Schematic on that board would have pushed those
references onto the copper and left three footprints called J73, against a
silkscreen that is already manufactured. The board is physical reality, so
the schematic was back-annotated from it, values included: R 5K became 5K,
C 470nF became 470nF and so on, which is also the better BOM text.
Schematic parity on that board goes from 6 to 0.

Backlighting_LEDModule had the same problem on one symbol, J73 -> J11.

The Korry resistors had no value in either schematic. Set to the fitted
parts, in the schematics and on the boards: RG 220 ohm for the green
annunciator, RW 91 ohm for the white backlight LED. At 5 V that is about
11 mA and 21 mA.

Three findings are deliberately left as they are, and the Readme now says
why rather than listing them as things to do:

- the dangling terminal block footprint has no replacement in KiCad 10,
  which ships no 2-pin 5.08 mm terminal block. Retargeting it would change
  the pads of a board already made
- the unmirrored + and - markers on the Korry_Large back silkscreen are
  symmetric glyphs, so nothing reads wrong, and mirroring them would move
  them sideways
- the PWR_FLAG the LEDModule wants is a two-click job in Eeschema. That
  file is KiCad 8 and the symbol definition would have to come from a
  KiCad 10 library carrying five toke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
Parts:
- renumbered J73 to J11
Changed lines of the file:
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@@
 		(dnp no)
 		(fields_autoplaced yes)
-		(property "Reference" "J73"
+		(property "Reference" "J11"
 			(at 72.39 140.97 0)
 			(effects
@@
 			(project "FCU_Mainboard_v2"
 				(path "/3267b3f3-6c63-480a-8354-1757ed0a4fd3/7ac51fd7-f93f-468f-8c10-b814dd9f4aef"
-					(reference "J73")
+					(reference "J11")
 					(unit 1)
 				)

Commit message: Put +5V on pin 1 of the LEDModule input
Il dimmer ha il +5V sul pin 1 di tutte e tre le sue uscite; il LEDModule ce
l'aveva sul pin 2 del suo ingresso, e su J11 non c'era nessun segno a dirlo.
Da qui il cavetto incrociato: dritto, i LED bianchi si trovano polarizzati
al contrario e non si accendono affatto.

La scheda non ha componenti e ha due soli nodi, N1 (J11 pin 1 piu' le file
dispari) e N2 (J11 pin 2 piu' le pari), quindi il rame non si tocca: bastano
i due nomi di rete e le lettere '+' e '-' che marcano le file. N1 diventa il
+5V marcato '+', e da li' in poi va tutto dritto, dal dimmer fino al Korry.

Aggiunti un '+' e un '-' sopra al contorno di J11, che era nudo ed e' la
ragione per cui ci si sbaglia.

La classe di rete +9V non corrispondeva a nessuna rete; ora e' +5V, cosi'
tutte e due le reti hanno gli 0.8 mm con cui sono gia' disegnate.

Netlist: J11 pin 1 = +5V, file dispari = +5V. ERC e DRC invariati, restano
solo gli avvisi di libreria che c'erano gia'.

Attenzione al montaggio: le schede fatte con questi file vogliono i tre
cavetti dal dimmer DRITTI, non incrociati.

Co-Authored-By: Claude Opus 5 <noreply@anthropic.com>
Connections:
- net +5V: now also J1.1 (Pin_1), J1.11 (Pin_11), J1.13 (Pin_13), J1.15 (Pin_15), J1.17 (Pin_17), J1.19 (Pin_19), J1.3 (Pin_3), J1.5 (Pin_5), J1.7 (Pin_7), J1.9 (Pin_9), J11.1 (Pin_1), J2.1 (Pin_1), J2.11 (Pin_11), J2.13 (Pin_13), J2.15 (Pin_15), J2.17 (Pin_17), J2.19 (Pin_19), J2.3 (Pin_3), J2.5 (Pin_5), J2.7 (Pin_7), J2.9 (Pin_9); no longer J1.10 (Pin_10), J1.12 (Pin_12), J1.14 (Pin_14), J1.16 (Pin_16), J1.18 (Pin_18), J1.2 (Pin_2), J1.20 (Pin_20), J1.4 (Pin_4), J1.6 (Pin_6), J1.8 (Pin_8), J11.2 (Pin_2), J2.10 (Pin_10), J2.12 (Pin_12), J2.14 (Pin_14), J2.16 (Pin_16), J2.18 (Pin_18), J2.2 (Pin_2), J2.20 (Pin_20), J2.4 (Pin_4), J2.6 (Pin_6), J2.8 (Pin_8)
- net GND: now also J1.10 (Pin_10), J1.12 (Pin_12), J1.14 (Pin_14), J1.16 (Pin_16), J1.18 (Pin_18), J1.2 (Pin_2), J1.20 (Pin_20), J1.4 (Pin_4), J1.6 (Pin_6), J1.8 (Pin_8), J11.2 (Pin_2), J2.10 (Pin_10), J2.12 (Pin_12), J2.14 (Pin_14), J2.16 (Pin_16), J2.18 (Pin_18), J2.2 (Pin_2), J2.20 (Pin_20), J2.4 (Pin_4), J2.6 (Pin_6), J2.8 (Pin_8); no longer J1.1 (Pin_1), J1.11 (Pin_11), J1.13 (Pin_13), J1.15 (Pin_15), J1.17 (Pin_17), J1.19 (Pin_19), J1.3 (Pin_3), J1.5 (Pin_5), J1.7 (Pin_7), J1.9 (Pin_9), J11.1 (Pin_1), J2.1 (Pin_1), J2.11 (Pin_11), J2.13 (Pin_13), J2.15 (Pin_15), J2.17 (Pin_17), J2.19 (Pin_19), J2.3 (Pin_3), J2.5 (Pin_5), J2.7 (Pin_7), J2.9 (Pin_9)
Changed lines of the file:
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@@
 	)
 	(symbol
-		(lib_id "power:+5V")
+		(lib_id "power:GND")
 		(at 77.47 124.46 180)
 		(unit 1)
@@
 			)
 		)
-		(property "Value" "+5V"
+		(property "Value" "GND"
 			(at 77.47 131.572 90)
 			(show_name no)
@@
 	)
 	(symbol
-		(lib_id "power:GND")
+		(lib_id "power:+5V")
 		(at 25.4 124.46 0)
 		(unit 1)
@@
 			)
 		)
-		(property "Value" "GND"
+		(property "Value" "+5V"
 			(at 25.4 129.54 0)
 			(show_name no)
@@
 	)
 	(symbol
-		(lib_id "power:GND")
+		(lib_id "power:+5V")
 		(at 62.23 140.97 270)
 		(unit 1)
@@
 			)
 		)
-		(property "Value" "GND"
+		(property "Value" "+5V"
 			(at 58.42 140.9699 90)
 			(show_name no)
@@
 	)
 	(symbol
-		(lib_id "power:GND")
+		(lib_id "power:+5V")
 		(at 55.88 124.46 0)
 		(unit 1)
@@
 			)
 		)
-		(property "Value" "GND"
+		(property "Value" "+5V"
 			(at 55.88 129.54 0)
 			(show_name no)
@@
 	)
 	(symbol
-		(lib_id "power:+5V")
+		(lib_id "power:GND")
 		(at 46.99 124.46 180)
 		(unit 1)
@@
 			)
 		)
-		(property "Value" "+5V"
+		(property "Value" "GND"
 			(at 46.99 131.572 90)
 			(show_name no)
@@
 	)
 	(symbol
-		(lib_id "power:+5V")
+		(lib_id "power:GND")
 		(at 62.23 143.51 90)
 		(unit 1)
@@
 			)
 		)
-		(property "Value" "+5V"
+		(property "Value" "GND"
 			(at 55.118 143.51 90)
 			(show_name no)

Commit message: Use the same terminal block everywhere
Le due schede backlighting stavano su TerminalBlock_bornier-2_P5.08mm, che
la libreria KiCad 10 non ha piu'. Il morsetto e' lo stesso che sta su PSU e
mainboard, quindi ora lo e' anche nei file: Phoenix PT-1,5-2-5.0-H, su
J12, J13, J14 e J32 del dimmer e su J11 del LEDModule.

Cosa cambia nel rame: passo 5.08 -> 5.00, pad 3.0 -> 2.6, foro 1.52 -> 1.30.
Gli 8 centesimi di passo non li sente nessuno; il foro piu' stretto e' la
misura giusta per quel morsetto.

Il corpo Phoenix e' pero' 1.64 mm piu' profondo del bornier, e questo si
sente:
 - J12, J13 e J14 arrivavano a 0.04 mm dal courtyard dei fori di fissaggio.
   Alzati di un decimo;
 - J32 e J11 stavano a filo del bordo scheda col vecchio corpo e col nuovo
   sporgevano. Rientrati, J11 esattamente dove stava prima la sua faccia
   esterna;
 - le estremita' delle piste sono state riagganciate ai nuovi centri dei
   pad, 13 in tutto, invece di lasciarle fuori centro;
 - le tre scritte TO LEDMODULE non ci stavano piu' sopra ai morsetti: una
   sola sotto alla fila, che sono tre uscite identiche.

Resta un solo avviso sul dimmer, ed e' geometria, non una svista: il
disegno dell'imbocco filo di J32 sfiora il bordo scheda a 0.02 mm. Per
rientrare J32 dovrebbe scendere, ma sotto ha C4 a 0.04 mm dal suo
courtyard: la finestra utile e' alta 10.49 mm per un corpo da 10. Tenuto
l'errore di courtyard risolto e lasciato l'avviso serigrafico, che vuol dire
solo che un pezzetto di inchiostro viene tagliato al bordo.

I problemi noti sono ora vuoti. Le zone delle due schede sono da riempire.

Co-Authored-By: Claude Opus 5 <noreply@anthropic.com>
Parts:
- J11: footprint TerminalBlock:TerminalBlock_bornier-2_P5.08mm -> TerminalBlock_Phoenix:TerminalBlock_Phoenix_PT-1,5-2-5.0-H_1x02_P5.00mm_Horizontal
Changed lines of the file:
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@@
 			)
 		)
-		(property "Footprint" "TerminalBlock:TerminalBlock_bornier-2_P5.08mm"
+		(property "Footprint" "TerminalBlock_Phoenix:TerminalBlock_Phoenix_PT-1,5-2-5.0-H_1x02_P5.00mm_Horizontal"
 			(at 69.85 140.97 0)
 			(hide yes)
