File: Korry_Small/KorrySmallPCB_SMD.kicad_pcb (KiCad board)
At the start: 2 copper layers, 22 x 36.7 mm, 9 parts, among them J1 BTN+LED, J2 BK_LED, SW1 SW

Commit message: Fix the swapped EFIS filenames and rename the backlight nets to +5V
Two naming defects, no electrical change on any board.

EFIS sheets
-----------
The root sheet pointed EFIS_LEFT at efis_right.kicad_sch and EFIS_RIGHT at
efis_left.kicad_sch. The schematic was correct, since the file behind the
LEFT sheet did hold the L_* signals, but the filenames said the opposite and
anyone reading the files from outside KiCad would have been misled.

The two files are swapped and every reference follows: the sheet properties
in the root schematic and the 49 sheetfile entries the footprints carry on
the board. Each file now matches the sheet that loads it.

  netlist   198 nets, 135 components, not one node moved
  ERC       0 violations
  DRC       6 violations, all cosmetic, 0 unconnected, 0 parity issues

Backlight nets
--------------
Every net in the backlighting chain was called +9V while carrying 5 V, on
all four boards. The white LEDs sit behind 91 Ω: at 5 V that is 21 mA, right
at the rating for a 1206 white LED, while 9 V would put them at 65 mA. The
name was a leftover from an earlier design and was the kind of label that
eventually makes someone connect the wrong supply.

Renamed across Korry_Large, Korry_Small, Backlighting_Dimmer and
Backlighting_LEDModule, in both the schematics and the boards: the power
symbol, its value, which is what actually names the net, and the net entries
on the copper. 88 occurrences. None of those boards had a +5V net already,
so nothing was merged.

Verified against the state committed a moment ago: ERC and DRC counts are
identical on all four boards, before and after, and no board gained or lost
a connection.

The Readme drops these two entries and gains the defects that surfaced while
checking: the Backlighting_Dimmer footprints carry their reference in the
value field instead of the schematic value, so a BOM read from that board is
wrong; its terminal block footprint no longer exists in the KiCad library;
four texts on the Korry_Large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
Connections:
- net +9V renamed +5V
Changed lines of the file:
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@@
 	)
 	(net 0 "")
-	(net 1 "+9V")
+	(net 1 "+5V")
 	(net 2 "/LED_INPUT")
 	(net 3 "GND")
@@
 			(layers "*.Cu" "*.Mask")
 			(remove_unused_layers no)
-			(net 1 "+9V")
+			(net 1 "+5V")
 			(pinfunction "Pin_1")
 			(pintype "passive")
@@
 			(layers "B.Cu" "B.Paste" "B.Mask")
 			(roundrect_rratio 0.175439)
-			(net 1 "+9V")
+			(net 1 "+5V")
 			(pinfunction "A")
 			(pintype "passive")

Commit message: Re-annotate the dimmer against its board, set the Korry resistor values
Tidying only. No board changed, no connection moved: all six projects still
report 0 unconnected items and 0 schematic parity issues.

Backlighting_Dimmer was worse than the value mismatch the Readme recorded.
Its schematic and its board disagreed on six reference designators, and
three separate connectors in the schematic all carried J73:

  J73 -> J12, J13, J14     three connectors sharing one reference
  J12 -> J31               J12 was the potentiometer in the schematic and a
                           terminal block on the board
  J93 -> J32
  U2  -> U1

Running Update PCB from Schematic on that board would have pushed those
references onto the copper and left three footprints called J73, against a
silkscreen that is already manufactured. The board is physical reality, so
the schematic was back-annotated from it, values included: R 5K became 5K,
C 470nF became 470nF and so on, which is also the better BOM text.
Schematic parity on that board goes from 6 to 0.

Backlighting_LEDModule had the same problem on one symbol, J73 -> J11.

The Korry resistors had no value in either schematic. Set to the fitted
parts, in the schematics and on the boards: RG 220 ohm for the green
annunciator, RW 91 ohm for the white backlight LED. At 5 V that is about
11 mA and 21 mA.

Three findings are deliberately left as they are, and the Readme now says
why rather than listing them as things to do:

- the dangling terminal block footprint has no replacement in KiCad 10,
  which ships no 2-pin 5.08 mm terminal block. Retargeting it would change
  the pads of a board already made
- the unmirrored + and - markers on the Korry_Large back silkscreen are
  symmetric glyphs, so nothing reads wrong, and mirroring them would move
  them sideways
- the PWR_FLAG the LEDModule wants is a two-click job in Eeschema. That
  file is KiCad 8 and the symbol definition would have to come from a
  KiCad 10 library carrying five toke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
Parts:
- RG-1: value R -> 220
- RW-1: value R -> 91
Changed lines of the file:
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@@
 			)
 		)
-		(property "Value" "R"
+		(property "Value" "91"
 			(at 0 1.82 0)
 			(layer "F.Fab")
@@
 			)
 		)
-		(property "Value" "R"
+		(property "Value" "220"
 			(at 0 1.82 0)
 			(layer "F.Fab")

Commit message: Align the Korry connector with the mainboard
La mainboard mette GND sul pin 1 di tutti e 34 i suoi connettori a 3 pin. I
Korry avevano pin 1 = pulsante e pin 3 = GND, quindi con un cavetto dritto
la massa finiva sull'ingresso del pulsante e l'ingresso del multiplexer
sulla massa del Korry. Funzionava solo infilando il connettore al
contrario.

Scambiati i pin 1 e 3 sul Korry, che ha un connettore per scheda, e non
sulla mainboard, che ne ha venti e che con GND sul pin 1 e' coerente con se
stessa.

Sullo schema il simbolo di J1 e' specchiato sull'asse X: i pin 1 e 3 si
scambiano di posto e i fili che c'erano finiscono da soli su quello giusto.
Sul rame si sono scambiate le reti dei due pad e si e' rifatta la pista del
pulsante, che ora esce dall'altro capo del connettore; la massa la prende il
piano come prima. Sul Korry grande la pista scansa il pad 3 dello switch,
che e' massa e sta in mezzo.

Scambiate anche le lettere 'G' e 'B' sul serigrafico, che indicano i pin e
sarebbero diventate bugiarde.

Netlist verificata: J1 ora e' 1=GND, 2=LED_INPUT, 3=BTN_INPUT su entrambe.
Le zone sono da riempire.

Co-Authored-By: Claude Opus 5 <noreply@anthropic.com>
Connections:
- J1 pad 1: /BTN_INPUT -> GND
- J1 pad 3: GND -> /BTN_INPUT
Routing:
- net /BTN_INPUT: track 18.6 -> 22.5 mm
Changed lines of the file:
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@@
 			(layers "*.Cu" "*.Mask")
 			(remove_unused_layers no)
-			(net "/BTN_INPUT")
+			(net "GND")
 			(pinfunction "Pin_1")
 			(pintype "passive")
@@
 			(layers "*.Cu" "*.Mask")
 			(remove_unused_layers no)
-			(net "GND")
+			(net "/BTN_INPUT")
 			(pinfunction "Pin_3")
 			(pintype "passive")
@@
 		)
 	)
-	(gr_text "G"
+	(gr_text "B"
 		(at 77.75 16.75 0)
 		(layer "F.SilkS")
@@
 		)
 	)
-	(gr_text "B"
+	(gr_text "G"
 		(at 77.75 22 0)
 		(layer "F.SilkS")
@@
 	)
 	(segment
-		(start 72.1 26.4)
-		(end 75.36 29.66)
-		(width 0.25)
-		(layer "F.Cu")
-		(net "/BTN_INPUT")
-	)
-	(segment
-		(start 75.36 29.66)
-		(end 75.36 33.2)
-		(width 0.25)
-		(layer "F.Cu")
-		(net "/BTN_INPUT")
-	)
-	(segment
 		(start 74.91 33.65)
 		(end 72.28 33.65)
@@
 		(start 75.36 33.2)
 		(end 74.91 33.65)
-		(width 0.25)
-		(layer "F.Cu")
-		(net "/BTN_INPUT")
-	)
-	(segment
-		(start 76.35 20.95)
-		(end 72.1 25.2)
-		(width 0.25)
-		(layer "F.Cu")
-		(net "/BTN_INPUT")
-	)
-	(segment
-		(start 72.1 25.2)
-		(end 72.1 26.4)
 		(width 0.25)
 		(layer "F.Cu")
@@
 	)
 	(embedded_fonts no)
+	(segment
+		(start 76.35 15.87)
+		(end 78.2 17.72)
+		(width 0.25)
+		(layer "F.Cu")
+		(net "/BTN_INPUT")
+	)
+	(segment
+		(start 78.2 17.72)
+		(end 78.2 30.36)
+		(width 0.25)
+		(layer "F.Cu")
+		(net "/BTN_INPUT")
+	)
+	(segment
+		(start 78.2 30.36)
+		(end 75.36 33.2)
+		(width 0.25)
+		(layer "F.Cu")
+		(net "/BTN_INPUT")
+	)
 )

Commit message: Call the 5 V rail 5 V on the boards that only ever see 5 V
Il Korry piccolo e il dimmer portavano ancora riferimenti a una rete +9V che
su quelle schede non esiste: entrambe sono alimentate a 5 V dal buck della
PSU.

Korry piccolo: la serigrafia accanto al pin 1 di J2 diceva "+9" ed e' il pin
del +5V. La classe di rete si chiamava 9V e il suo pattern cercava +9V, cioe'
non prendeva niente, mentre i suoi 0.75 mm sono esattamente la larghezza con
cui la rete +5V e' gia' disegnata: era solo il nome a essere sbagliato.

Dimmer: il pattern della classe PowerLine cercava +9V invece di +5V, e anche
il colore di rete era assegnato a +9V. I suoi 1.5 mm sono, di nuovo, la
larghezza con cui +5V e' gia' disegnata.

Tutte le classi coinvolte hanno la stessa distanza di isolamento del
Default, 0.2 mm, quindi rimettere a posto i pattern non puo' introdurre
violazioni: cambia solo la larghezza di default per il routing futuro.
Verificato, DRC invariato su entrambe.

Sulla PSU il riferimento a +9V resta, perche' quella scheda i 9 V li porta
davvero.

Co-Authored-By: Claude Opus 5 <noreply@anthropic.com>
Other:
- board text added: "+5"
- board text removed: "+9"
Changed lines of the file:
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@@
 		)
 	)
-	(gr_text "+9"
+	(gr_text "+5"
 		(at 57.5 18 0)
 		(layer "F.SilkS")
@@
 	)
 	(segment
-		(start 59.5 37.03)
-		(end 59.54 36.99)
-		(width 0.75)
-		(layer "B.Cu")
-		(net "+5V")
-	)
-	(segment
-		(start 59.5 37.03)
-		(end 59.56 36.97)
-		(width 0.75)
-		(layer "B.Cu")
-		(net "+5V")
-	)
-	(segment
-		(start 62.275 17.1)
-		(end 59.5 19.875)
-		(width 0.75)
-		(layer "B.Cu")
-		(net "+5V")
-	)
-	(segment
-		(start 66.58 36.99)
-		(end 67.575 36.99)
-		(width 0.75)
-		(layer "B.Cu")
-		(net "+5V")
-	)
-	(segment
-		(start 67.575 36.99)
-		(end 67.625 36.94)
-		(width 0.75)
-		(layer "B.Cu")
-		(net "+5V")
-	)
-	(segment
-		(start 59.54 36.99)
-		(end 67.405 36.99)
-		(width 0.75)
-		(layer "B.Cu")
-		(net "+5V")
-	)
-	(segment
-		(start 59.5 19.875)
-		(end 59.5 37.03)
-		(width 0.75)
-		(layer "B.Cu")
-		(net "+5V")
-	)
-	(segment
-		(start 70.75 24.01)
-		(end 70.75 30.34)
-		(width 0.25)
-		(layer "B.Cu")
-		(net "/LED_INPUT")
-	)
-	(segment
-		(start 70.75 30.34)
-		(end 70.7 30.39)
-		(width 0.25)
-		(layer "B.Cu")
-		(net "/LED_INPUT")
-	)
-	(segment
-		(start 76.35 18.41)
-		(end 70.75 24.01)
-		(width 0.25)
-		(layer "B.Cu")
-		(net "/LED_INPUT")
-	)
-	(segment
-		(start 74.91 33.65)
-		(end 72.28 33.65)
-		(width 0.25)
-		(layer "F.Cu")
-		(net "/BTN_INPUT")
-	)
-	(segment
-		(start 75.36 33.2)
-		(end 74.91 33.65)
-		(width 0.25)
-		(layer "F.Cu")
-		(net "/BTN_INPUT")
-	)
-	(segment
 		(start 69 40.35)
 		(end 74.4 45.75)
@@
 		(layer "F.Cu")
 		(net "/LED_PCB")
+	)
+	(segment
+		(start 77.6 44.6)
+		(end 74.25 41.25)
+		(width 0.8)
+		(layer "F.Cu")
+		(net "Net-(DW-1-K)")
+	)
+	(segment
+		(start 77.6 45.75)
+		(end 77.6 44.6)
+		(width 0.8)
+		(layer "F.Cu")
+		(net "Net-(DW-1-K)")
+	)
+	(via
+		(at 74.25 41.25)
+		(size 0.8)
+		(drill 0.4)
+		(layers "F.Cu" "B.Cu")
+		(capping no)
+		(covering
+			(front no)
+			(back no)
+		)
+		(plugging
+			(front no)
+			(back no)
+		)
+		(filling no)
+		(net "Net-(DW-1-K)")
+	)
+	(segment
+		(start 74.25 41.25)
+		(end 70.38 37.38)
+		(width 0.8)
+		(layer "B.Cu")
+		(net "Net-(DW-1-K)")
+	)
+	(segment
+		(start 70.43 36.94)
+		(end 70.6 36.94)
+		(width 0.8)
+		(layer "B.Cu")
+		(net "Net-(DW-1-K)")
+	)
+	(segment
+		(start 70.38 37.38)
+		(end 70.38 36.99)
+		(width 0.8)
+		(layer "B.Cu")
+		(net "Net-(DW-1-K)")
+	)
+	(segment
+		(start 70.38 36.99)
+		(end 70.43 36.94)
+		(width 0.8)
+		(layer "B.Cu")
+		(net "Net-(DW-1-K)")
 	)
 	(segment
@@
 	)
 	(segment
-		(start 77.6 44.6)
-		(end 74.25 41.25)
-		(width 0.8)
-		(layer "F.Cu")
-		(net "Net-(DW-1-K)")
-	)
-	(segment
-		(start 77.6 45.75)
-		(end 77.6 44.6)
-		(width 0.8)
-		(layer "F.Cu")
-		(net "Net-(DW-1-K)")
-	)
-	(via
-		(at 74.25 41.25)
-		(size 0.8)
-		(drill 0.4)
-		(layers "F.Cu" "B.Cu")
-		(capping no)
-		(covering
-			(front no)
-			(back no)
-		)
-		(plugging
-			(front no)
-			(back no)
-		)
-		(filling no)
-		(net "Net-(DW-1-K)")
-	)
-	(segment
-		(start 74.25 41.25)
-		(end 70.38 37.38)
-		(width 0.8)
-		(layer "B.Cu")
-		(net "Net-(DW-1-K)")
-	)
-	(segment
-		(start 70.43 36.94)
-		(end 70.6 36.94)
-		(width 0.8)
-		(layer "B.Cu")
-		(net "Net-(DW-1-K)")
-	)
-	(segment
-		(start 70.38 37.38)
-		(end 70.38 36.99)
-		(width 0.8)
-		(layer "B.Cu")
-		(net "Net-(DW-1-K)")
-	)
-	(segment
-		(start 70.38 36.99)
-		(end 70.43 36.94)
-		(width 0.8)
-		(layer "B.Cu")
-		(net "Net-(DW-1-K)")
+		(start 59.5 37.03)
+		(end 59.54 36.99)
+		(width 0.75)
+		(layer "B.Cu")
+		(net "+5V")
+	)
+	(segment
+		(start 59.5 37.03)
+		(end 59.56 36.97)
+		(width 0.75)
+		(layer "B.Cu")
+		(net "+5V")
+	)
+	(segment
+		(start 62.275 17.1)
+		(end 59.5 19.875)
+		(width 0.75)
+		(layer "B.Cu")
+		(net "+5V")
+	)
+	(segment
+		(start 66.58 36.99)
+		(end 67.575 36.99)
+		(width 0.75)
+		(layer "B.Cu")
+		(net "+5V")
+	)
+	(segment
+		(start 67.575 36.99)
+		(end 67.625 36.94)
+		(width 0.75)
+		(layer "B.Cu")
+		(net "+5V")
+	)
+	(segment
+		(start 59.54 36.99)
+		(end 67.405 36.99)
+		(width 0.75)
+		(layer "B.Cu")
+		(net "+5V")
+	)
+	(segment
+		(start 59.5 19.875)
+		(end 59.5 37.03)
+		(width 0.75)
+		(layer "B.Cu")
+		(net "+5V")
+	)
+	(segment
+		(start 70.75 24.01)
+		(end 70.75 30.34)
+		(width 0.25)
+		(layer "B.Cu")
+		(net "/LED_INPUT")
+	)
+	(segment
+		(start 70.75 30.34)
+		(end 70.7 30.39)
+		(width 0.25)
+		(layer "B.Cu")
+		(net "/LED_INPUT")
+	)
+	(segment
+		(start 76.35 18.41)
+		(end 70.75 24.01)
+		(width 0.25)
+		(layer "B.Cu")
+		(net "/LED_INPUT")
+	)
+	(segment
+		(start 76.35 15.87)
+		(end 78.2 17.72)
+		(width 0.25)
+		(layer "F.Cu")
+		(net "/BTN_INPUT")
+	)
+	(segment
+		(start 74.91 33.65)
+		(end 72.28 33.65)
+		(width 0.25)
+		(layer "F.Cu")
+		(net "/BTN_INPUT")
+	)
+	(segment
+		(start 78.2 17.72)
+		(end 78.2 30.36)
+		(width 0.25)
+		(layer "F.Cu")
+		(net "/BTN_INPUT")
+	)
+	(segment
+		(start 78.2 30.36)
+		(end 75.36 33.2)
+		(width 0.25)
+		(layer "F.Cu")
+		(net "/BTN_INPUT")
+	)
+	(segment
+		(start 75.36 33.2)
+		(end 74.91 33.65)
+		(width 0.25)
+		(layer "F.Cu")
+		(net "/BTN_INPUT")
 	)
 	(zone
@@
 	)
 	(embedded_fonts no)
-	(segment
-		(start 76.35 15.87)
-		(end 78.2 17.72)
-		(width 0.25)
-		(layer "F.Cu")
-		(net "/BTN_INPUT")
-	)
-	(segment
-		(start 78.2 17.72)
-		(end 78.2 30.36)
-		(width 0.25)
-		(layer "F.Cu")
-		(net "/BTN_INPUT")
-	)
-	(segment
-		(start 78.2 30.36)
-		(end 75.36 33.2)
-		(width 0.25)
-		(layer "F.Cu")
-		(net "/BTN_INPUT")
-	)
 )

Commit message: Say on the silkscreen what plugs into each connector
Le schede da fabbricate non si leggevano: quasi tutti i valori stavano su
F.Fab, che non va in stampa, e meta' dei connettori aveva come nome il tipo
di morsetto invece di cosa ci va attaccato.

Nessun valore e' stato riscritto: il nome del componente resta quello che
dice KiCad. Si e' lavorato solo sul serigrafico, in due modi.

I valori che gia' dicono qualcosa di utile sono passati su F.Silk, cosi' si
stampano: Backlighting POT sul dimmer, BTN+LED e BK_LED sui Korry, e i 220 e
91 delle due resistenze, che da montare sono due rettangoli identici.

Dove il valore e' il tipo di morsetto e stampalo non servirebbe a niente, il
valore resta dov'e' e accanto ci va una scritta che dice dove va il filo:

  PSU        J1 -> 9V IN, J2/J3/J4 -> 5V BACKLIGHT, J5 -> 5V MAINBOARD
  Dimmer     J32 -> 5V IN, J12/J13/J14 -> TO LEDMODULE
  LEDModule  J11 -> 5V IN

Ogni posizione e' stata verificata contro pad, altre scritte, contorni
serigrafici e bordo scheda, e poi ricontrollata col DRC, che e' l'unico a
sapere quanto e' larga davvero l'apertura di maschera di un foro di
fissaggio: la scritta di J14 ci finiva sopra, e il valore di J1 sul Korry
grande finiva a cavallo del bordo.

Tutte e cinque le schede: 0 scollegamenti, 0 differenze con lo schema,
nessuna violazione serigrafica. Restano solo gli avvisi di libreria.

Co-Authored-By: Claude Opus 5 <noreply@anthropic.com>
Changed lines of the file:
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@@
 		(property "Value" "91"
 			(at 0 1.82 0)
-			(layer "F.Fab")
+			(layer "F.SilkS")
 			(effects
 				(font
@@
 		(property "Value" "220"
 			(at 0 1.82 0)
-			(layer "F.Fab")
+			(layer "F.SilkS")
 			(effects
 				(font

Commit message: Update the last three boards from the library
Aggiornati i footprint di LEDModule, Korry grande e Korry piccolo, come era
gia' stato fatto sul dimmer. Le quattordici lib_footprint_mismatch che
restavano sono chiuse.

Le serigrafie hanno retto anche qui: 220, 91, BK_LED e BTN+LED sono ancora
su F.Silk su tutti e due i Korry, e tutte le scritte libere sono al loro
posto. Piste e posizioni dei componenti invariate: 128, 28 e 28 tratti,
stessi estremi e stesse larghezze.

L'aggiornamento ha allargato di poco il contorno di J2 sul Korry piccolo, e
la scritta '+5' arrivava a 0.09 mm da esso. A sinistra non poteva andare,
perche' partiva gia' 0.15 mm fuori dal bordo scheda: e' diventata '+', e per
coerenza la 'L' dell'altro piolo e' diventata '-'. Ora quel connettore e'
marcato come quello del Korry grande e come le file del LEDModule.

Nota per la prossima volta: il font a tratti di KiCad avanza circa 1.0 em
per carattere, non 0.72 come stimava il mio controllo. Per questo un paio di
scritte che avevo dato per libere sono poi state prese dal DRC.

Co-Authored-By: Claude Opus 5 <noreply@anthropic.com>
Other:
- board text added: "-"
- board text removed: "+5"
